Commit message: Task 1.3 & 1.4 : Fix bugs in desherborator_materials desherborator_parameters desherborator_sensor

File: desherborator_description/urdf/desherborator.materials.xacro (robot description, xacro)
@@ -1,6 +1,6 @@
-<xml version="1.0"?>
+<?xml version="1.0"?>
 <!-- Here are defined the materials used for defining the robot in the simulation
     Author : Elodie NOELE -->
-<robot>
+<robot name="desherborator_materials" xmlns:xacro="http://ros.org/wiki/xacro">
   <material name="black">
     <color rgba="0.0 0.0 0.0 1.0"/>

File: desherborator_description/urdf/desherborator.parameters.xacro (robot description, xacro)
@@ -1,4 +1,4 @@
 <?xml version="1.0"?>
-<robot name="desherborator" xmlns:xacro="http://www.ros.org/wiki/xacro">
+<robot name="desherborator_parametors" xmlns:xacro="http://www.ros.org/wiki/xacro">
     <xacro:property name="chassisHeight" value="0.2"/>
     <xacro:property name="chassisWidth" value="0.3"/>

File: desherborator_description/urdf/desherborator.sensor.xacro (robot description, xacro)
@@ -1,3 +1,3 @@
-<xml version="1.0"?>
+<?xml version="1.0"?>
 <!-- Create the robot sensors. The robot has the following sensors :
     Lidar : an hokuyo sensor
@@ -5,9 +5,9 @@
     Laser : the laser for burning the weeds
     Author : Elodie NOELE -->
-<xacro:include filename="./desherborator.parameters.xacro" />
-<xacro:include filename="./desherborator.materials.xacro" />
-<xacro:include filename="./desherborator.joint.xacro" />
-<xacro:property name="chassisHeight" value="0.1"/>
-<robot name="desherborator" xmlns:xacro="http://ros.org/wiki/xacro">
+<robot name="desherborator_sensor" xmlns:xacro="http://ros.org/wiki/xacro">
+    <xacro:include filename="./desherborator.parameters.xacro" />
+    <xacro:include filename="./desherborator.materials.xacro" />
+    <xacro:include filename="./desherborator.joint.xacro" />
+    <xacro:property name="chassisHeight" value="0.1"/>
     <xacro:macro name="LIDAR">
         <gazebo reference="LIDAR">
