Commit message: try it

File: desherborator_description/urdf/desherborator.link.xacro (robot description, xacro)
@@ -1,3 +1,4 @@
-<?xml version="1.0"?>
+<?xml version="1.0" encoding="UTF-8"?>
+<robot name="desherborator_links" xmlns:xacro="http://ros.org/wiki/xacro">
 <!-- ########################################################### -->
 <!-- #                link base_link                           # -->
@@ -161,5 +162,5 @@
 <link name="BrasC2">
 <collision>
-  <origin xyz="0 0 0" rpy="0 0 1.5707 1.5707"/>
+  <origin xyz="0 0 0" rpy="0 1.5707 1.5707"/>
   <geometry>
     <cylinder radius="0.01" length="0.3"/>
@@ -174,5 +175,5 @@
 </visual>
 <inertial>
-  <origin xyz="0 0 0" rpy="0 0 1.5707 1.5707"/>
+  <origin xyz="0 0 0" rpy="0 1.5707 1.5707"/>
   <mass value="0.01"/>
   <inertia
@@ -254,2 +255,3 @@
 </inertial>
 </link>
+</robot>

Commit message: fixed some issues

File: desherborator_description/urdf/desherborator.link.xacro (robot description, xacro)
@@ -1,10 +1,11 @@
-<?xml version="1.0"?>
-<!-- ########################################################### -->
-<!-- #                link base_link                           # -->
-<!-- ########################################################### -->
+<?xml version="1.0" encoding="UTF-8"?>
+<robot name="desherborator_links" xmlns:xacro="http://ros.org/wiki/xacro">
+<!-- #########################################################e# -->
+<!-- #                link base_link                          r# -->
+<!-- #########################################################r# -->
 <link name="base_link"/>
-<!-- ########################################################### -->
-<!-- #                link Chassis                             # -->
-<!-- ########################################################### -->
+<!-- #########################################################e# -->
+<!-- #                link Chassis                            u# -->
+<!-- #########################################################r# -->
 <link name="Chassis">
 <collision>
@@ -30,7 +31,7 @@
 </inertial>
 </link>
-<!-- ########################################################### -->
-<!-- #                link Roues                               # -->
-<!-- ########################################################### -->
+<!-- #########################################################t# -->
+<!-- #                link Roues                              r# -->
+<!-- #########################################################o# -->
 <!-- link Roue Folle -->
 <link name="RoueF">
@@ -105,7 +106,7 @@
 </inertial>
 </link>
-<!-- ########################################################### -->
-<!-- #                link Mat                                 # -->
-<!-- ########################################################### -->
+<!-- #########################################################v# -->
+<!-- #                link Mat                                é# -->
+<!-- #########################################################e# -->
 <link name="Mat">
 <collision>
@@ -131,7 +132,7 @@
 </inertial>
 </link>
-<!-- ########################################################### -->
-<!-- #                link Bras                                # -->
-<!-- ########################################################### -->
+<!-- ########################################################è é# -->
+<!-- #                link Bras                              /"\# -->
+<!-- ###################################################1####\_/# -->
 <!-- link Bras Cylindre 1 -->
 <link name="BrasC1">
@@ -161,5 +162,5 @@
 <link name="BrasC2">
 <collision>
-  <origin xyz="0 0 0" rpy="0 0 1.5707 1.5707"/>
+  <origin xyz="0 0 0" rpy="0 1.5707 1.5707"/>
   <geometry>
     <cylinder radius="0.01" length="0.3"/>
@@ -174,5 +175,5 @@
 </visual>
 <inertial>
-  <origin xyz="0 0 0" rpy="0 0 1.5707 1.5707"/>
+  <origin xyz="0 0 0" rpy="0 1.5707 1.5707"/>
   <mass value="0.01"/>
   <inertia
@@ -254,2 +255,3 @@
 </inertial>
 </link>
+</robot>

Commit message: Task 1.25 : Restore the right version

File: desherborator_description/urdf/desherborator.link.xacro (robot description, xacro)
@@ -1,257 +1,247 @@
-<?xml version="1.0" encoding="UTF-8"?>
+<?xml version="1.0"?>
 <robot name="desherborator_links" xmlns:xacro="http://ros.org/wiki/xacro">
-<!-- #########################################################e# -->
-<!-- #                link base_link                          r# -->
-<!-- #########################################################r# -->
-<link name="base_link"/>
-<!-- #########################################################e# -->
-<!-- #                link Chassis                            u# -->
-<!-- #########################################################r# -->
-<link name="Chassis">
-<collision>
-  <origin xyz="0 0 0.05" rpy="0 0 0"/>
-  <geometry>
-    <box size="0.4 0.3 0.2"/>
-  </geometry>
-</collision>
-<visual>
-  <origin xyz="0 0 0.05" rpy="0 0 0"/>
-  <geometry>
-    <box size="0.4 0.3 0.2"/>
-  </geometry>
-  <material name="black"/>
-</visual>
-<inertial>
-  <origin xyz="0 0 0.05" rpy="0 0 0"/>
-  <mass value="1"/>
-  <inertia
-    ixx="0.01" ixy="0.0" ixz="0.0"
-    iyy="0.01" iyz="0.0"
-    izz="0.01"/>
-</inertial>
-</link>
-<!-- #########################################################t# -->
-<!-- #                link Roues                              r# -->
-<!-- #########################################################o# -->
-<!-- link Roue Folle -->
-<link name="RoueF">
-<collision>
-  <origin xyz="0 0 0" rpy="0 0 0"/>
-  <geometry>
-    <sphere radius="0.05"/>
-  </geometry>
-</collision>
-<visual>
-  <origin xyz="0 0 0" rpy="0 0 0"/>
-  <geometry>
-    <sphere radius="0.05"/>
-  </geometry>
-  <material name="black"/>
-</visual>
-<inertial>
-  <origin xyz="0 0 0" rpy="0 0 0"/>
-  <mass value="0.01"/>
-  <inertia
-    ixx="0.01" ixy="0.0" ixz="0.0"
-    iyy="0.01" iyz="0.0"
-    izz="0.01"/>
-</inertial>
-</link>
-<!-- link Roue Gauche -->
-<link name="RoueG">
-<collision>
-  <origin xyz="0 0 0" rpy="0 1.5707 1.5707"/>
-  <geometry>
-    <cylinder radius="0.15" length="0.1"/>
-  </geometry>
-</collision>
-<visual>
-  <origin xyz="0 0 0" rpy="0 1.5707 1.5707"/>
-  <geometry>
-    <cylinder radius="0.15" length="0.1"/>
-  </geometry>
-  <material name="black"/>
-</visual>
-<inertial>
-  <origin xyz="0 0 0" rpy="0 0 0"/>
-  <mass value="0.01"/>
-  <inertia
-    ixx="0.01" ixy="0.0" ixz="0.0"
-    iyy="0.01" iyz="0.0"
-    izz="0.01"/>
-</inertial>
-</link>
-<!-- link Roue Droite -->
-<link name="RoueD">
-<collision>
-  <origin xyz="0 0 0" rpy="0 1.5707 1.5707"/>
-  <geometry>
-    <cylinder radius="0.15" length="0.1"/>
-  </geometry>
-</collision>
-<visual>
-  <origin xyz="0 0 0" rpy="0 1.5707 1.5707"/>
-  <geometry>
-    <cylinder radius="0.15" length="0.1"/>
-  </geometry>
-  <material name="black"/>
-</visual>
-<inertial>
-  <origin xyz="0 0 0" rpy="0 0 0"/>
-  <mass value="0.01"/>
-  <inertia
-    ixx="0.01" ixy="0.0" ixz="0.0"
-    iyy="0.01" iyz="0.0"
-    izz="0.01"/>
-</inertial>
-</link>
-<!-- #########################################################v# -->
-<!-- #                link Mat                                é# -->
-<!-- #########################################################e# -->
-<link name="Mat">
-<collision>
-  <origin xyz="0 0 0" rpy="0 0 0"/>
-  <geometry>
-    <cylinder radius="0.01" length="0.2"/>
-  </geometry>
-</collision>
-<visual>
-  <origin xyz="0 0 0" rpy="0 0 0"/>
-  <geometry>
-    <cylinder radius="0.01" length="0.2"/>
-  </geometry>
-  <material name="black"/>
-</visual>
-<inertial>
-  <origin xyz="0 0 0" rpy="0 0 0"/>
-  <mass value="0.01"/>
-  <inertia
-    ixx="0.01" ixy="0.0" ixz="0.0"
-    iyy="0.01" iyz="0.0"
-    izz="0.01"/>
-</inertial>
-</link>
-<!-- ########################################################è é# -->
-<!-- #                link Bras                              /"\# -->
-<!-- ###################################################1####\_/# -->
-<!-- link Bras Cylindre 1 -->
-<link name="BrasC1">
-<collision>
-  <origin xyz="0 0 0" rpy="0 0 0"/>
-  <geometry>
-    <cylinder radius="0.01" length="0.25"/>
-  </geometry>
-</collision>
-<visual>
-  <origin xyz="0 0 0" rpy="0 0 0"/>
-  <geometry>
-    <cylinder radius="0.01" length="0.25"/>
-  </geometry>
-  <material name="black"/>
-</visual>
-<inertial>
-  <origin xyz="0 0 0" rpy="0 0 0"/>
-  <mass value="0.01"/>
-  <inertia
-    ixx="0.01" ixy="0.0" ixz="0.0"
-    iyy="0.01" iyz="0.0"
-    izz="0.01"/>
-</inertial>
-</link>
-<!-- link Bras Cylindre 2 -->
-<link name="BrasC2">
-<collision>
-  <origin xyz="0 0 0" rpy="0 1.5707 1.5707"/>
-  <geometry>
-    <cylinder radius="0.01" length="0.3"/>
-  </geometry>
-</collision>
-<visual>
-  <origin xyz="0 0 0" rpy="0 0 0"/>
-  <geometry>
-    <cylinder radius="0.01" length="0.3"/>
-  </geometry>
-  <material name="black"/>
-</visual>
-<inertial>
-  <origin xyz="0 0 0" rpy="0 1.5707 1.5707"/>
-  <mass value="0.01"/>
-  <inertia
-    ixx="0.01" ixy="0.0" ixz="0.0"
-    iyy="0.01" iyz="0.0"
-    izz="0.01"/>
-</inertial>
-</link>
-<!-- link Bras Cylindre 3 -->
-<link name="BrasC3">
-<collision>
-  <origin xyz="0 0 0" rpy="0 3.14 0"/>
-  <geometry>
-    <cylinder radius="0.01" length="0.1"/>
-  </geometry>
-</collision>
-<visual>
-  <origin xyz="0 0 0" rpy="0 3.14 0"/>
-  <geometry>
-    <cylinder radius="0.01" length="0.1"/>
-  </geometry>
-  <material name="black"/>
-</visual>
-<inertial>
-  <origin xyz="0 0 0" rpy="0 0 0"/>
-  <mass value="0.01"/>
-  <inertia
-    ixx="0.01" ixy="0.0" ixz="0.0"
-    iyy="0.01" iyz="0.0"
-    izz="0.01"/>
-</inertial>
-</link>
-<!-- link Bras Sphere 1 -->
-<link name="BrasS1">
-<collision>
-  <origin xyz="0 0 0" rpy="0 0 0"/>
-  <geometry>
-    <sphere radius="0.02"/>
-  </geometry>
-</collision>
-<visual>
-  <origin xyz="0 0 0" rpy="0 0 0"/>
-  <geometry>
-    <sphere radius="0.02"/>
-  </geometry>
-  <material name="black"/>
-</visual>
-<inertial>
-  <origin xyz="0 0 0" rpy="0 0 0"/>
-  <mass value="0.01"/>
-  <inertia
-    ixx="0.01" ixy="0.0" ixz="0.0"
-    iyy="0.01" iyz="0.0"
-    izz="0.01"/>
-</inertial>
-</link>
-<!-- link Bras Sphere 2 -->
-<link name="BrasS2">
-<collision>
-  <origin xyz="0 0 0" rpy="0 0 0"/>
-  <geometry>
-    <sphere radius="0.02"/>
-  </geometry>
-</collision>
-<visual>
-  <origin xyz="0 0 0" rpy="0 0 0"/>
-  <geometry>
-    <sphere radius="0.02"/>
-  </geometry>
-  <material name="black"/>
-</visual>
-<inertial>
-  <origin xyz="0 0 0" rpy="0 0 0"/>
-  <mass value="0.01"/>
-  <inertia
-    ixx="0.01" ixy="0.0" ixz="0.0"
-    iyy="0.01" iyz="0.0"
-    izz="0.01"/>
-</inertial>
-</link>
+  <!-- Base Chassis -->
+  <link name="base_link"/>
+  <!-- Link Chassis -->
+  <link name="Chassis">
+  <collision>
+    <origin xyz="0 0 0.05" rpy="0 0 0"/>
+    <geometry>
+      <box size="0.4 0.3 0.2"/>
+    </geometry>
+  </collision>
+  <visual>
+    <origin xyz="0 0 0.05" rpy="0 0 0"/>
+    <geometry>
+      <box size="0.4 0.3 0.2"/>
+    </geometry>
+    <material name="black"/>
+  </visual>
+  <inertial>
+    <origin xyz="0 0 0.05" rpy="0 0 0"/>
+    <mass value="1"/>
+    <inertia
+      ixx="0.01" ixy="0.0" ixz="0.0"
+      iyy="0.01" iyz="0.0"
+      izz="0.01"/>
+  </inertial>
+  </link>
+  <!-- Link Roue -->
+  <!-- link Roue Folle -->
+  <link name="RoueF">
+  <collision>
+    <origin xyz="0 0 0" rpy="0 0 0"/>
+    <geometry>
+      <sphere radius="0.05"/>
+    </geometry>
+  </collision>
+  <visual>
+    <origin xyz="0 0 0" rpy="0 0 0"/>
+    <geometry>
+      <sphere radius="0.05"/>
+    </geometry>
+    <material name="black"/>
+  </visual>
+  <inertial>
+    <origin xyz="0 0 0" rpy="0 0 0"/>
+    <mass value="0.01"/>
+    <inertia
+      ixx="0.01" ixy="0.0" ixz="0.0"
+      iyy="0.01" iyz="0.0"
+      izz="0.01"/>
+  </inertial>
+  </link>
+  <!-- link Roue Gauche -->
+  <link name="RoueG">
+  <collision>
+    <origin xyz="0 0 0" rpy="0 1.5707 1.5707"/>
+    <geometry>
+      <cylinder radius="0.15" length="0.1"/>
+    </geometry>
+  </collision>
+  <visual>
+    <origin xyz="0 0 0" rpy="0 1.5707 1.5707"/>
+    <geometry>
+      <cylinder radius="0.15" length="0.1"/>
+    </geometry>
+    <material name="black"/>
+  </visual>
+  <inertial>
+    <origin xyz="0 0 0" rpy="0 0 0"/>
+    <mass value="0.01"/>
+    <inertia
+      ixx="0.01" ixy="0.0" ixz="0.0"
+      iyy="0.01" iyz="0.0"
+      izz="0.01"/>
+  </inertial>
+  </link>
+  <!-- link Roue Droite -->
+  <link name="RoueD">
+  <collision>
+    <origin xyz="0 0 0" rpy="0 1.5707 1.5707"/>
+    <geometry>
+      <cylinder radius="0.15" length="0.1"/>
+    </geometry>
+  </collision>
+  <visual>
+    <origin xyz="0 0 0" rpy="0 1.5707 1.5707"/>
+    <geometry>
+      <cylinder radius="0.15" length="0.1"/>
+    </geometry>
+    <material name="black"/>
+  </visual>
+  <inertial>
+    <origin xyz="0 0 0" rpy="0 0 0"/>
+    <mass value="0.01"/>
+    <inertia
+      ixx="0.01" ixy="0.0" ixz="0.0"
+      iyy="0.01" iyz="0.0"
+      izz="0.01"/>
+  </inertial>
+  </link>
+  <!-- link Mat -->
+  <link name="Mat">
+  <collision>
+    <origin xyz="0 0 0" rpy="0 0 0"/>
+    <geometry>
+      <cylinder radius="0.01" length="0.2"/>
+    </geometry>
+  </collision>
+  <visual>
+    <origin xyz="0 0 0" rpy="0 0 0"/>
+    <geometry>
+      <cylinder radius="0.01" length="0.2"/>
+    </geometry>
+    <material name="black"/>
+  </visual>
+  <inertial>
+    <origin xyz="0 0 0" rpy="0 0 0"/>
+    <mass value="0.01"/>
+    <inertia
+      ixx="0.01" ixy="0.0" ixz="0.0"
+      iyy="0.01" iyz="0.0"
+      izz="0.01"/>
+  </inertial>
+  </link>
+  <!-- link Bras -->
+  <!-- link Bras Cylindre 1 -->
+  <link name="BrasC1">
+  <collision>
+    <origin xyz="0 0 0" rpy="0 0 0"/>
+    <geometry>
+      <cylinder radius="0.01" length="0.25"/>
+    </geometry>
+  </collision>
+  <visual>
+    <origin xyz="0 0 0" rpy="0 0 0"/>
+    <geometry>
+      <cylinder radius="0.01" length="0.25"/>
+    </geometry>
+    <material name="black"/>
+  </visual>
+  <inertial>
+    <origin xyz="0 0 0" rpy="0 0 0"/>
+    <mass value="0.01"/>
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
File: desherborator_description/urdf/desherborator.urdf.xacro (robot description, xacro)
@@ -2,7 +2,7 @@
 <robot name="desherborator" xmlns:xacro="http://ros.org/wiki/xacro">
   <xacro:include filename="$(find desherborator_description)/urdf/desherborator.joint.xacro"/>
-  <!--<xacro:include filename="$(find desherborator_description)/urdf/desherborator.link.xacro"/>
+  <xacro:include filename="$(find desherborator_description)/urdf/desherborator.link.xacro"/>
+  <xacro:include filename="$(find desherborator_description)/urdf/desherborator.sensor.xacro"/>
   <xacro:include filename="$(find desherborator_description)/urdf/desherborator.materials.xacro"/>
-  <xacro:include filename="$(find desherborator_description)/urdf/desherborator.sensor.xacro"/>
-    -->
+  <xacro:include filename="$(find desherborator_description)/urdf/desherborator.parameters.xacro"/>
 </robot>
