Commit message: Task 2.10 & 4.8 : Fix colors in Gazebo and Add controllers for wheels

File: desherborator_description/urdf/desherborator.controller.xacro (robot description, xacro)
@@ -9,5 +9,5 @@
       <publishOdomTF>true</publishOdomTF>
       <!-- ENTER BASE LINK NAME -->
-      <robotBaseFrame>Chassis</robotBaseFrame>
+      <robotBaseFrame>base_link</robotBaseFrame>
       <publishWheelTF>true</publishWheelTF>
       <publishTf>true</publishTf>
@@ -16,7 +16,7 @@
       <updateRate>30</updateRate>
       <!-- ENTER LEFT JOINT NAME -->
-      <leftJoint>joint_2</leftJoint>
+      <leftJoint>joint_chassis_to_roueG</leftJoint>
       <!-- ENTER RIGHT JOINT NAME -->
-      <rightJoint>joint_1</rightJoint>
+      <rightJoint>joint_chassis_to_roueD</rightJoint>
       <wheelSeparation>0.31</wheelSeparation>
       <wheelDiameter>0.1</wheelDiameter>

File: desherborator_description/urdf/desherborator.joint.xacro (robot description, xacro)
@@ -4,60 +4,59 @@
                 <parent link="base_link"/>
                 <child link="Chassis"/>
-                <origin xyz="0 0 0.05" rpy="0 0 0"/>
+                <origin xyz="0 0 0.2" rpy="0 0 0"/>
         </joint>
         <joint name="mat_attached" type="fixed">
                 <parent link="Chassis"/>
                 <child link="Mat"/>
-                <origin xyz="-0.3 0 0.2" rpy="0 0 0"/>
+                <origin xyz="0.1 0 0.3" rpy="0 0 0"/>
         </joint>
-        <joint name="joint_1" type="continuous">
+        <joint name="joint_chassis_to_roueD" type="continuous">
                 <parent link="Chassis"/>
                 <child link="RoueD"/>
-                <origin xyz="-0.2 -0.15 0.1" rpy="0 0 0"/>
+                <origin xyz="0.1 -0.15 0.1" rpy="0 0 0"/>
                 <axis  xyz="0 1 0"/>
         </joint>
-        <joint name="joint_2" type="continuous">
+        <joint name="joint_chassis_to_roueG" type="continuous">
                 <parent link="Chassis"/>
                 <child link="RoueG"/>
-                <origin xyz="-0.2 0.15 0.1" rpy="0 0 0"/>
+                <origin xyz="0.1 0.15 0.1" rpy="0 0 0"/>
                 <axis  xyz="0 1 0"/>
         </joint>
-        <joint name="joint_3" type="fixed">
+        <joint name="joint_chassis_to_roueF" type="fixed">
                 <parent link="Chassis"/>
                 <child link="RoueF"/>
-                <origin xyz="-0.3 0 0" rpy="0 0 0"/>
+                <origin xyz="-0.10 0 0" rpy="0 0 0"/>
         </joint>
-        <joint name="joint_4" type="continuous">
+        <joint name="joint_chassis_to_dummy" type="fixed">
                 <parent link="Chassis"/>
                 <child link="BrasC1dummy"/>
-                <origin xyz="0.01 -0.15 0" rpy="0 0 0"/>
+                <origin xyz="0.19 -0.06 0.2" rpy="0 0 0"/>
                 <axis  xyz="0 0 1"/>
         </joint>
-        <joint name="joint_5" type="prismatic">
+        <joint name="joint_dummy_to_rotating_bras" type="fixed">
                 <parent link="BrasC1dummy"/>
                 <child link="BrasC1"/>
-                <origin xyz="0 0 0.01" rpy="0 0 0"/>
+                <origin xyz="0 0 0" rpy="0 0 0"/>
                 <axis  xyz="0 0 1"/>
-                <limit  lower="0"  upper="0.10"  effort="10"  velocity="1"/>
         </joint>
-        <joint name="joint_6" type="fixed">
+        <joint name="joint_rotating_bras_to_brasS" type="fixed">
                 <parent link="BrasC1"/>
                 <child link="BrasS1"/>
-                <origin xyz="0 0 0.10" rpy="0 0 0"/>
+                <origin xyz="0 0 0.11" rpy="0 0 0"/>
         </joint>
-        <joint name="joint_7" type="fixed">
+        <joint name="joint_brasS_to_brasC" type="fixed">
                 <parent link="BrasS1"/>
                 <child link="BrasC2"/>
-                <origin xyz="0 0 0" rpy="0  0  0"/>
+                <origin xyz="0 0.15 0" rpy="0  0  0"/>
         </joint>
-        <joint name="joint_8" type="fixed">
+        <joint name="joint_brasC_to_brasS" type="fixed">
                 <parent link="BrasC2"/>
                 <child link="BrasS2"/>
-                <origin xyz="0 0.3 0" rpy="0 0 0"/>
+                <origin xyz="0 0.15 0" rpy="0 0 0"/>
         </joint>
-        <joint name="joint_9" type="fixed">
+        <joint name="end_joint" type="fixed">
                 <parent link="BrasS2"/>
                 <child link="BrasC3"/>
-                <origin xyz="0 0 0" rpy="0 0 0"/>
+                <origin xyz="0 0 -0.05" rpy="0 0 0"/>
         </joint>
 </robot>

File: desherborator_description/urdf/desherborator.link.xacro (robot description, xacro)
@@ -6,5 +6,5 @@
   <link name="Chassis">
     <collision>
-      <origin xyz="0 0 0.05" rpy="0 0 0"/>
+      <origin xyz="0 0 .1" rpy="0 0 0"/>
       <geometry>
         <box size="0.4 0.3 0.2"/>
@@ -12,17 +12,10 @@
     </collision>
     <visual>
-      <origin xyz="0 0 0.05" rpy="0 0 0"/>
+      <origin xyz="0 0 .1" rpy="0 0 0"/>
       <geometry>
         <box size="0.4 0.3 0.2"/>
       </geometry>
     </visual>
-    <inertial>
-      <origin xyz="0 0 0.05" rpy="0 0 0"/>
-      <mass value="1"/>
-      <inertia
-        ixx="0.01" ixy="0.0" ixz="0.0"
-        iyy="0.01" iyz="0.0"
-        izz="0.01"/>
-    </inertial>
+    <xacro:default_inertial mass="2.0"/>
   </link>
   <!-- Link Roue -->
@@ -41,12 +34,5 @@
       </geometry>
     </visual>
-    <inertial>
-      <origin xyz="0 0 0" rpy="0 0 0"/>
-      <mass value="0.01"/>
-      <inertia
-        ixx="0.01" ixy="0.0" ixz="0.0"
-        iyy="0.01" iyz="0.0"
-        izz="0.01"/>
-    </inertial>
+    <xacro:default_inertial mass="0.01"/>
   </link>
   <!-- link Roue Gauche -->
@@ -64,12 +50,5 @@
       </geometry>
     </visual>
-    <inertial>
-      <origin xyz="0 0 0" rpy="0 0 0"/>
-      <mass value="0.01"/>
-      <inertia
-        ixx="0.01" ixy="0.0" ixz="0.0"
-        iyy="0.01" iyz="0.0"
-        izz="0.01"/>
-    </inertial>
+    <xacro:default_inertial mass="0.3"/>
   </link>
   <!-- link Roue Droite -->
@@ -87,17 +66,10 @@
       </geometry>
     </visual>
-    <inertial>
-      <origin xyz="0 0 0" rpy="0 0 0"/>
-      <mass value="0.01"/>
-      <inertia
-        ixx="0.01" ixy="0.0" ixz="0.0"
-        iyy="0.01" iyz="0.0"
-        izz="0.01"/>
-    </inertial>
+    <xacro:default_inertial mass="0.3"/>
   </link>
   <!-- link Mat -->
   <link name="Mat">
     <collision>
-      <origin xyz="0 0 0" rpy="0 0 0"/>
+      <origin xyz="0.1 0 0.3" rpy="0 0 0"/>
       <geometry>
         <cylinder radius="0.01" length="0.2"/>
@@ -110,12 +82,5 @@
       </geometry>
     </visual>
-    <inertial>
-      <origin xyz="0 0 0" rpy="0 0 0"/>
-      <mass value="0.01"/>
-      <inertia
-        ixx="0.01" ixy="0.0" ixz="0.0"
-        iyy="0.01" iyz="0.0"
-        izz="0.01"/>
-    </inertial>
+    <xacro:default_inertial mass="0.1"/>
   </link>
   <!-- link Bras -->
@@ -134,12 +99,5 @@
     </geometry>
   </visual>
-  <inertial>
-    <origin xyz="0 0 0" rpy="0 0 0"/>
-    <mass value="0.01"/>
-    <inertia
-      ixx="0.01" ixy="0.0" ixz="0.0"
-      iyy="0.01" iyz="0.0"
-      izz="0.01"/>
-  </inertial>
+    <xacro:default_inertial mass="0.1"/>
   </link>
   <!-- link Dummy Bras Cylindre 1 -->
@@ -148,5 +106,5 @@
   <link name="BrasC2">
     <collision>
-      <origin xyz="0 0 0" rpy="0 1.5707 1.5707"/>
+      <origin xyz="0 0 0" rpy="0 ${PI/2} ${PI/2}"/>
       <geometry>
         <cylinder radius="0.01" length="0.3"/>
@@ -154,22 +112,15 @@
     </collision>
     <visual>
-      <origin xyz="0 0 0" rpy="0 0 0"/>
+      <origin xyz="0 0 0" rpy="0 ${PI/2} ${PI/2}"/>
       <geometry>
         <cylinder radius="0.01" length="0.3"/>
       </geometry>
     </visual>
-    <inertial>
-      <origin xyz="0 0 0" rpy="0 1.5707 1.5707"/>
-      <mass value="0.01"/>
-      <inertia
-        ixx="0.01" ixy="0.0" ixz="0.0"
-        iyy="0.01" iyz="0.0"
-        izz="0.01"/>
-    </inertial>
+    <xacro:default_inertial mass="0.01"/>
   </link>
   <!-- link Bras Cylindre 3 -->
   <link name="BrasC3">
     <collision>
-      <origin xyz="0 0 0" rpy="0 3.14 0"/>
+      <origin xyz="0 0 0" rpy="0 ${PI} 0"/>
       <geometry>
         <cylinder radius="0.01" length="0.1"/>
@@ -177,17 +128,10 @@
     </collision>
     <visual>
-      <origin xyz="0 0 0" rpy="0 3.14 0"/>
+      <origin xyz="0 0 0" rpy="0 ${PI} 0"/>
       <geometry>
         <cylinder radius="0.01" length="0.1"/>
       </geometry>
     </visual>
-    <inertial>
-      <origin xyz="0 0 0" rpy="0 0 0"/>
-      <mass value="0.01"/>
-      <inertia
-        ixx="0.01" ixy="0.0" ixz="0.0"
-        iyy="0.01" iyz="0.0"
-        izz="0.01"/>
-    </inertial>
+    <xacro:default_inertial mass="0.01"/>
   </link>
   <!-- link Bras Sphere 1 -->
@@ -205,12 +149,5 @@
       </geometry>
     </visual>
-    <inertial>
-      <origin xyz="0 0 0" rpy="0 0 0"/>
-      <mass value="0.01"/>
-      <inertia
-        ixx="0.01" ixy="0.0" ixz="0.0"
-        iyy="0.01" iyz="0.0"
-        izz="0.01"/>
-    </inertial>
+    <xacro:default_inertial mass="0.01"/>
   </link>
   <!-- link Bras Sphere 2 -->
@@ -228,12 +165,5 @@
       </geometry>
     </visual>
-    <inertial>
-      <origin xyz="0 0 0" rpy="0 0 0"/>
-      <mass value="0.01"/>
-      <inertia
-        ixx="0.01" ixy="0.0" ixz="0.0"
-        iyy="0.01" iyz="0.0"
-        izz="0.01"/>
-    </inertial>
+    <xacro:default_inertial mass="0.01"/>
   </link>
 </robot>

File: desherborator_description/urdf/desherborator.materials.xacro (robot description, xacro)
@@ -13,5 +13,5 @@
     <minDepth>0.001</minDepth>
     <maxVel>0.1</maxVel>
-    <material>Gazebo/FlatBlack</material>
+    <material>Gazebo/Purple</material>
   </gazebo>
   <gazebo reference="RoueD">
@@ -22,5 +22,5 @@
     <minDepth>0.001</minDepth>
     <maxVel>0.1</maxVel>
-    <material>Gazebo/FlatBlack</material>
+    <material>Gazebo/Purple</material>
   </gazebo>
   <gazebo reference="RoueF">
@@ -31,23 +31,23 @@
     <minDepth>0.001</minDepth>
     <maxVel>1.0</maxVel>
-    <material>Gazebo/FlatBlack</material>
+    <material>Gazebo/Purple</material>
   </gazebo>
   <gazebo reference="Mat">
-    <material>Gazebo/FlatBlack</material>
+    <material>Gazebo/Orange</material>
   </gazebo>
   <gazebo reference="BrasC1">
-    <material>Gazebo/FlatBlack</material>
+    <material>Gazebo/Turquoise</material>
   </gazebo>
   <gazebo reference="BrasC2">
-    <material>Gazebo/FlatBlack</material>
+    <material>Gazebo/Turquoise</material>
   </gazebo>
   <gazebo reference="BrasC3">
-    <material>Gazebo/FlatBlack</material>
+    <material>Gazebo/Turquoise</material>
   </gazebo>
   <gazebo reference="BrasS1">
-    <material>Gazebo/FlatBlack</material>
+    <material>Gazebo/Turquoise</material>
   </gazebo>
   <gazebo reference="BrasS2">
-    <material>Gazebo/FlatBlack</material>
+    <material>Gazebo/Turquoise</material>
   </gazebo>
 </robot>

File: desherborator_description/urdf/desherborator.parameters.xacro (robot description, xacro)
@@ -2,8 +2,9 @@
 <robot name="desherborator" xmlns:xacro="http://ros.org/wiki/xacro">
     <xacro:property name="ChassisHeight" value="0.2"/>
-    <xacro:property name="ChassisWidth" value="0.3"/>
+    <xacro:property name="ChassisWidth" value="0.2"/>
     <xacro:property name="cameraSize" value="0.1"/>
     <xacro:property name="wheelRadius" value="0.15"/>
     <xacro:property name="wheelWidth" value="0.1"/>
+    <xacro:property name="PI" value="3.1459"/>
     <xacro:macro name="default_inertial" params="mass">
         <inertial>

File: desherborator_description/urdf/desherborator.sensor.xacro (robot description, xacro)
@@ -11,7 +11,7 @@
     </link>
     <joint name="lidar_joint" type="fixed">
-        <parent link="Chassis"/>
+        <parent link="Mat"/>
         <child link="LIDAR"/>
-        <origin xyz="0.15 0 0.23" rpy="0 0 0"/>
+        <origin xyz="0 0 0.075" rpy="0 0 0"/>
     </joint>
     <gazebo reference="LIDAR">
@@ -27,5 +27,5 @@
                 <resolution>1</resolution>
                 <min_angle>0.0</min_angle>
-                <max_angle>6.28319</max_angle>
+                <max_angle>6.2</max_angle>
             </horizontal>
             </scan>
@@ -42,5 +42,5 @@
         </ray>
         <plugin name="gazebo_ros_lds_lfcd_controller" filename="libgazebo_ros_laser.so">
-            <topicName>laser_scan</topicName>
+            <topicName>/laser_scan</topicName>
             <!-- ENTER FRAME NAME -->
             <frameName>LIDAR</frameName>
@@ -50,6 +50,6 @@
     <joint name="camera_joint" type="fixed">
         <parent link="Chassis"/>
-        <axis xyz="0 0 0" />
-        <origin xyz="${ChassisWidth} 0 ${ChassisHeight/2}" rpy="0 0 0"/>
+        <axis xyz="0 1 0" />
+        <origin xyz="${ChassisWidth} 0 ${ChassisHeight/2}" rpy="0 ${PI/2} 0"/>
         <child link="Camera"/>
     </joint>
@@ -124,7 +124,7 @@
     </link>
     <joint name="laser_joint" type="fixed">
-        <parent link="Chassis"/>
+        <parent link="BrasC3"/>
         <child link="LASER"/>
-        <origin xyz="0.15 0 0.23" rpy="0 0 0"/>
+        <origin xyz="0 0 0" rpy="0 ${PI/2} 0"/>
     </joint>
     <gazebo reference="LASER">
@@ -137,5 +137,5 @@
             <scan>
             <horizontal>
-                <samples>720</samples>
+                <samples>10</samples>
                 <resolution>1</resolution>
                 <min_angle>0.0</min_angle>
@@ -155,7 +155,7 @@
         </ray>
         <plugin name="gazebo_ros_lds_lfcd_controller" filename="libgazebo_ros_laser.so">
-            <topicName>laser</topicName>
+            <topicName>/laser</topicName>
             <!-- ENTER FRAME NAME -->
-            <frameName>laser</frameName>
+            <frameName>LASER</frameName>
         </plugin>
         </sensor>

File: desherborator_description/urdf/desherborator.urdf (robot description, URDF)
Before this commit: robot desherborator, 15 links, 14 joints
Links:
- link BrasC1: mass 0.01 -> 0.1
- link Chassis: mass 1 -> 2.0
- link Mat: mass 0.01 -> 0.1
- link RoueD: mass 0.01 -> 0.3
- link RoueG: mass 0.01 -> 0.3
Joints:
- removed joint joint_1
- removed joint joint_2
- removed joint joint_3
- removed joint joint_4
- removed joint joint_5
- removed joint joint_6
- removed joint joint_7
- removed joint joint_8
- removed joint joint_9
- added joint end_joint: type fixed, parent BrasS2, child BrasC3, origin xyz=0 0 -0.05 rpy=0 0 0
- added joint joint_brasC_to_brasS: type fixed, parent BrasC2, child BrasS2, origin xyz=0 0.15 0 rpy=0 0 0
- added joint joint_brasS_to_brasC: type fixed, parent BrasS1, child BrasC2, origin xyz=0 0.15 0 rpy=0  0  0
- added joint joint_chassis_to_dummy: type fixed, parent Chassis, child BrasC1dummy, origin xyz=0.19 -0.06 0.2 rpy=0 0 0, axis 0 0 1
- added joint joint_chassis_to_roueD: type continuous, parent Chassis, child RoueD, origin xyz=0.1 -0.15 0.1 rpy=0 0 0, axis 0 1 0
- added joint joint_chassis_to_roueF: type fixed, parent Chassis, child RoueF, origin xyz=-0.10 0 0 rpy=0 0 0
- added joint joint_chassis_to_roueG: type continuous, parent Chassis, child RoueG, origin xyz=0.1 0.15 0.1 rpy=0 0 0, axis 0 1 0
- added joint joint_dummy_to_rotating_bras: type fixed, parent BrasC1dummy, child BrasC1, origin xyz=0 0 0 rpy=0 0 0, axis 0 0 1
- added joint joint_rotating_bras_to_brasS: type fixed, parent BrasC1, child BrasS1, origin xyz=0 0 0.11 rpy=0 0 0
- joint base_joint: origin xyz=0 0 0.05 rpy=0 0 0 -> xyz=0 0 0.2 rpy=0 0 0
- joint camera_joint: axis 0 0 0 -> 0 1 0; origin xyz=0.3 0 0.1 rpy=0 0 0 -> xyz=0.2 0 0.1 rpy=0 1.57295 0
- joint laser_joint: origin xyz=0.15 0 0.23 rpy=0 0 0 -> xyz=0 0 0 rpy=0 1.57295 0; parent Chassis -> BrasC3
- joint lidar_joint: origin xyz=0.15 0 0.23 rpy=0 0 0 -> xyz=0 0 0.075 rpy=0 0 0; parent Chassis -> Mat
- joint mat_attached: origin xyz=-0.3 0 0.2 rpy=0 0 0 -> xyz=0.1 0 0.3 rpy=0 0 0
