Commit message: Maj pose camera

File: desherborator_description/urdf/desherborator.sensor.xacro (robot description, xacro)
@@ -51,5 +51,5 @@
         <parent link="Chassis"/>
         <axis xyz="0 1 0" />
-        <origin xyz="${ChassisWidth} 0 ${ChassisHeight/2}" rpy="0 ${PI/2} 0"/>
+        <origin xyz="${ChassisWidth} 0 ${ChassisHeight/2}" rpy="0 0 0"/>
         <child link="Camera"/>
     </joint>

Commit message: Task 2.42: Simulate GPS + noise

File: desherborator_description/urdf/desherborator.sensor.xacro (robot description, xacro)
@@ -161,3 +161,30 @@
         </sensor>
     </gazebo>
+    <link name="GPS_link">
+        <visual>
+        <origin xyz="0 0 0" rpy="0 0 0"/>
+        <geometry>
+            <cylinder radius="0.005" length="0.005"/>
+        </geometry>
+        </visual>
+        <xacro:default_inertial mass="0.05"/>
+    </link>
+    <joint name="GPS_joint" type="fixed">
+        <parent link="Chassis"/>
+        <child link="GPS_link"/>
+        <origin xyz="-0.01 0 0" rpy="0 0 0"/>
+    </joint>
+<gazebo>
+    <plugin filename="libhector_gazebo_ros_gps.so" name="GPS_link">
+        <alwayson>true</alwayson>
+        <updateRate>10</updateRate>
+        <bodyName>GPS_link</bodyName>
+        <topicName>/fix</topicName>
+        <velocityTopicName>/vel</velocityTopicName>
+        <drift>5.0 5.0 5.0</drift>
+        <gaussianNoise>0.0000001 0.0000001 0.0000001</gaussianNoise>
+        <velocityDrift>0 0 0</velocityDrift>
+        <velocityGaussianNoise>0.0000001 0.0000001 0.0000001</velocityGaussianNoise>
+    </plugin>
+</gazebo>
 </robot>
