Commit message: Fix bug when launching everything together

File: desherborator_description/urdf/desherborator.joint.xacro (robot description, xacro)
@@ -1,64 +1,63 @@
-<?xml  version="1.0"?>
-<robot  name="desherborator_joints"  xmlns:xacro="http://ros.org/wiki/xacro">
-        <xacro:include  filename="$(find  desherborator_description)/urdf/desherborator.link.xacro"/>
-        <joint  name="base_joint"  type="fixed">
-                <parent  link="base_link"/>
-                <child  link="Chassis"  />
-                <origin  xyz="0  0  0.05"  rpy="0  0  0"/>
+<?xml version="1.0"?>
+<robot name="desherborator_joints" xmlns:xacro="http://ros.org/wiki/xacro">
+        <joint name="base_joint" type="fixed">
+                <parent link="base_link"/>
+                <child link="Chassis"/>
+                <origin xyz="0 0 0.05" rpy="0 0 0"/>
         </joint>
-        <joint  name="mat_attached"  type="fixed">
-                <parent  link="Chassis"/>
-                <child  link="Mat"  />
-                <origin  xyz="-0.3  0  0.2"  rpy="0  0  0"/>
+        <joint name="mat_attached" type="fixed">
+                <parent link="Chassis"/>
+                <child link="Mat"/>
+                <origin xyz="-0.3 0 0.2" rpy="0 0 0"/>
         </joint>
-        <joint  name="joint_1"  type="continuous">
-                <parent  link="Chassis"/>
-                <child  link="RoueD"  />
-                <origin  xyz="-0.2  -0.15  0.1"  rpy="0  0  0"/>
-                <axis  xyz="0  1  0"/>
+        <joint name="joint_1" type="continuous">
+                <parent link="Chassis"/>
+                <child link="RoueD"/>
+                <origin xyz="-0.2 -0.15 0.1" rpy="0 0 0"/>
+                <axis  xyz="0 1 0"/>
         </joint>
-        <joint  name="joint_2"  type="continuous">
-                <parent  link="Chassis"/>
-                <child  link="RoueG"  />
-                <origin  xyz="-0.2  0.15  0.1"  rpy="0  0  0"/>
-                <axis  xyz="0  1  0"/>
+        <joint name="joint_2" type="continuous">
+                <parent link="Chassis"/>
+                <child link="RoueG"/>
+                <origin xyz="-0.2 0.15 0.1" rpy="0 0 0"/>
+                <axis  xyz="0 1 0"/>
         </joint>
-        <joint  name="joint_3"  type="fixed">
-                <parent  link="Chassis"/>
-                <child  link="RoueF"  />
-                <origin  xyz="-0.3  0  0"  rpy="0  0  0"/>
+        <joint name="joint_3" type="fixed">
+                <parent link="Chassis"/>
+                <child link="RoueF"/>
+                <origin xyz="-0.3 0 0" rpy="0 0 0"/>
         </joint>
-        <joint  name="joint_4"  type="continuous">
-                <parent  link="Chassis"/>
-                <child  link="BrasC1"  />
-                <origin  xyz="0.01  -0.15  0"  rpy="0  0  0"/>
-                <axis  xyz="0  0  1"/>
+        <joint name="joint_4" type="continuous">
+                <parent link="Chassis"/>
+                <child link="BrasC1"/>
+                <origin xyz="0.01 -0.15 0" rpy="0 0 0"/>
+                <axis  xyz="0 0 1"/>
         </joint>
-        <joint  name="joint_5"  type="prismatic">
-                <parent  link="Chassis"/>
-                <child  link="BrasC1"  />
-                <origin  xyz="0  0  0.01"  rpy="0  0  0"/>
-                <axis  xyz="0  0  1"/>
+        <joint name="joint_5" type="prismatic">
+                <parent link="Chassis"/>
+                <child link="BrasC1"/>
+                <origin xyz="0 0 0.01" rpy="0 0 0"/>
+                <axis  xyz="0 0 1"/>
                 <limit  lower="0"  upper="0.10"  effort="10"  velocity="1"/>
         </joint>
-        <joint  name="joint_6"  type="fixed">
-                <parent  link="BrasC1"/>
-                <child  link="BrasS1"  />
-                <origin  xyz="0  0  0.10"  rpy="0  0  0"/>
+        <joint name="joint_6" type="fixed">
+                <parent link="BrasC1"/>
+                <child link="BrasS1"/>
+                <origin xyz="0 0 0.10" rpy="0 0 0"/>
         </joint>
-        <joint  name="joint_7"  type="fixed">
-                <parent  link="BrasS1"/>
-                <child  link="BrasC2"  />
-                <origin  xyz="0  0  0"  rpy="0  0  0"/>
+        <joint name="joint_7" type="fixed">
+                <parent link="BrasS1"/>
+                <child link="BrasC2"/>
+                <origin xyz="0 0 0" rpy="0  0  0"/>
         </joint>
-        <joint  name="joint_8"  type="fixed">
-                <parent  link="BrasC2"/>
-                <child  link="BrasS2"  />
-                <origin  xyz="0  0.3  0"  rpy="0  0  0"/>
+        <joint name="joint_8" type="fixed">
+                <parent link="BrasC2"/>
+                <child link="BrasS2"/>
+                <origin xyz="0 0.3 0" rpy="0 0 0"/>
         </joint>
-        <joint  name="joint_9"  type="fixed">
-                <parent  link="BrasS2"/>
-                <child  link="BrasC3"  />
-                <origin  xyz="0  0  0"  rpy="0  0  0"/>
+        <joint name="joint_9" type="fixed">
+                <parent link="BrasS2"/>
+                <child link="BrasC3"/>
+                <origin xyz="0 0 0" rpy="0 0 0"/>
         </joint>
 </robot>

File: desherborator_description/urdf/desherborator.link.xacro (robot description, xacro)
@@ -1,257 +1,247 @@
-<?xml version="1.0" encoding="UTF-8"?>
+<?xml version="1.0"?>
 <robot name="desherborator_links" xmlns:xacro="http://ros.org/wiki/xacro">
-<!-- ########################################################### -->
-<!-- #                link base_link                           # -->
-<!-- ########################################################### -->
-<link name="base_link"/>
-<!-- ########################################################### -->
-<!-- #                link Chassis                             # -->
-<!-- ########################################################### -->
-<link name="Chassis">
-<collision>
-  <origin xyz="0 0 0.05" rpy="0 0 0"/>
-  <geometry>
-    <box size="0.4 0.3 0.2"/>
-  </geometry>
-</collision>
-<visual>
-  <origin xyz="0 0 0.05" rpy="0 0 0"/>
-  <geometry>
-    <box size="0.4 0.3 0.2"/>
-  </geometry>
-  <material name="black"/>
-</visual>
-<inertial>
-  <origin xyz="0 0 0.05" rpy="0 0 0"/>
-  <mass value="1"/>
-  <inertia
-    ixx="0.01" ixy="0.0" ixz="0.0"
-    iyy="0.01" iyz="0.0"
-    izz="0.01"/>
-</inertial>
-</link>
-<!-- ########################################################### -->
-<!-- #                link Roues                               # -->
-<!-- ########################################################### -->
-<!-- link Roue Folle -->
-<link name="RoueF">
-<collision>
-  <origin xyz="0 0 0" rpy="0 0 0"/>
-  <geometry>
-    <sphere radius="0.05"/>
-  </geometry>
-</collision>
-<visual>
-  <origin xyz="0 0 0" rpy="0 0 0"/>
-  <geometry>
-    <sphere radius="0.05"/>
-  </geometry>
-  <material name="black"/>
-</visual>
-<inertial>
-  <origin xyz="0 0 0" rpy="0 0 0"/>
-  <mass value="0.01"/>
-  <inertia
-    ixx="0.01" ixy="0.0" ixz="0.0"
-    iyy="0.01" iyz="0.0"
-    izz="0.01"/>
-</inertial>
-</link>
-<!-- link Roue Gauche -->
-<link name="RoueG">
-<collision>
-  <origin xyz="0 0 0" rpy="0 1.5707 1.5707"/>
-  <geometry>
-    <cylinder radius="0.15" length="0.1"/>
-  </geometry>
-</collision>
-<visual>
-  <origin xyz="0 0 0" rpy="0 1.5707 1.5707"/>
-  <geometry>
-    <cylinder radius="0.15" length="0.1"/>
-  </geometry>
-  <material name="black"/>
-</visual>
-<inertial>
-  <origin xyz="0 0 0" rpy="0 0 0"/>
-  <mass value="0.01"/>
-  <inertia
-    ixx="0.01" ixy="0.0" ixz="0.0"
-    iyy="0.01" iyz="0.0"
-    izz="0.01"/>
-</inertial>
-</link>
-<!-- link Roue Droite -->
-<link name="RoueD">
-<collision>
-  <origin xyz="0 0 0" rpy="0 1.5707 1.5707"/>
-  <geometry>
-    <cylinder radius="0.15" length="0.1"/>
-  </geometry>
-</collision>
-<visual>
-  <origin xyz="0 0 0" rpy="0 1.5707 1.5707"/>
-  <geometry>
-    <cylinder radius="0.15" length="0.1"/>
-  </geometry>
-  <material name="black"/>
-</visual>
-<inertial>
-  <origin xyz="0 0 0" rpy="0 0 0"/>
-  <mass value="0.01"/>
-  <inertia
-    ixx="0.01" ixy="0.0" ixz="0.0"
-    iyy="0.01" iyz="0.0"
-    izz="0.01"/>
-</inertial>
-</link>
-<!-- ########################################################### -->
-<!-- #                link Mat                                 # -->
-<!-- ########################################################### -->
-<link name="Mat">
-<collision>
-  <origin xyz="0 0 0" rpy="0 0 0"/>
-  <geometry>
-    <cylinder radius="0.01" length="0.2"/>
-  </geometry>
-</collision>
-<visual>
-  <origin xyz="0 0 0" rpy="0 0 0"/>
-  <geometry>
-    <cylinder radius="0.01" length="0.2"/>
-  </geometry>
-  <material name="black"/>
-</visual>
-<inertial>
-  <origin xyz="0 0 0" rpy="0 0 0"/>
-  <mass value="0.01"/>
-  <inertia
-    ixx="0.01" ixy="0.0" ixz="0.0"
-    iyy="0.01" iyz="0.0"
-    izz="0.01"/>
-</inertial>
-</link>
-<!-- ########################################################### -->
-<!-- #                link Bras                                # -->
-<!-- ########################################################### -->
-<!-- link Bras Cylindre 1 -->
-<link name="BrasC1">
-<collision>
-  <origin xyz="0 0 0" rpy="0 0 0"/>
-  <geometry>
-    <cylinder radius="0.01" length="0.25"/>
-  </geometry>
-</collision>
-<visual>
-  <origin xyz="0 0 0" rpy="0 0 0"/>
-  <geometry>
-    <cylinder radius="0.01" length="0.25"/>
-  </geometry>
-  <material name="black"/>
-</visual>
-<inertial>
-  <origin xyz="0 0 0" rpy="0 0 0"/>
-  <mass value="0.01"/>
-  <inertia
-    ixx="0.01" ixy="0.0" ixz="0.0"
-    iyy="0.01" iyz="0.0"
-    izz="0.01"/>
-</inertial>
-</link>
-<!-- link Bras Cylindre 2 -->
-<link name="BrasC2">
-<collision>
-  <origin xyz="0 0 0" rpy="0 1.5707 1.5707"/>
-  <geometry>
-    <cylinder radius="0.01" length="0.3"/>
-  </geometry>
-</collision>
-<visual>
-  <origin xyz="0 0 0" rpy="0 0 0"/>
-  <geometry>
-    <cylinder radius="0.01" length="0.3"/>
-  </geometry>
-  <material name="black"/>
-</visual>
-<inertial>
-  <origin xyz="0 0 0" rpy="0 1.5707 1.5707"/>
-  <mass value="0.01"/>
-  <inertia
-    ixx="0.01" ixy="0.0" ixz="0.0"
-    iyy="0.01" iyz="0.0"
-    izz="0.01"/>
-</inertial>
-</link>
-<!-- link Bras Cylindre 3 -->
-<link name="BrasC3">
-<collision>
-  <origin xyz="0 0 0" rpy="0 3.14 0"/>
-  <geometry>
-    <cylinder radius="0.01" length="0.1"/>
-  </geometry>
-</collision>
-<visual>
-  <origin xyz="0 0 0" rpy="0 3.14 0"/>
-  <geometry>
-    <cylinder radius="0.01" length="0.1"/>
-  </geometry>
-  <material name="black"/>
-</visual>
-<inertial>
-  <origin xyz="0 0 0" rpy="0 0 0"/>
-  <mass value="0.01"/>
-  <inertia
-    ixx="0.01" ixy="0.0" ixz="0.0"
-    iyy="0.01" iyz="0.0"
-    izz="0.01"/>
-</inertial>
-</link>
-<!-- link Bras Sphere 1 -->
-<link name="BrasS1">
-<collision>
-  <origin xyz="0 0 0" rpy="0 0 0"/>
-  <geometry>
-    <sphere radius="0.02"/>
-  </geometry>
-</collision>
-<visual>
-  <origin xyz="0 0 0" rpy="0 0 0"/>
-  <geometry>
-    <sphere radius="0.02"/>
-  </geometry>
-  <material name="black"/>
-</visual>
-<inertial>
-  <origin xyz="0 0 0" rpy="0 0 0"/>
-  <mass value="0.01"/>
-  <inertia
-    ixx="0.01" ixy="0.0" ixz="0.0"
-    iyy="0.01" iyz="0.0"
-    izz="0.01"/>
-</inertial>
-</link>
-<!-- link Bras Sphere 2 -->
-<link name="BrasS2">
-<collision>
-  <origin xyz="0 0 0" rpy="0 0 0"/>
-  <geometry>
-    <sphere radius="0.02"/>
-  </geometry>
-</collision>
-<visual>
-  <origin xyz="0 0 0" rpy="0 0 0"/>
-  <geometry>
-    <sphere radius="0.02"/>
-  </geometry>
-  <material name="black"/>
-</visual>
-<inertial>
-  <origin xyz="0 0 0" rpy="0 0 0"/>
-  <mass value="0.01"/>
-  <inertia
-    ixx="0.01" ixy="0.0" ixz="0.0"
-    iyy="0.01" iyz="0.0"
-    izz="0.01"/>
-</inertial>
-</link>
+  <!-- Base Chassis -->
+  <link name="base_link"/>
+  <!-- Link Chassis -->
+  <link name="Chassis">
+  <collision>
+    <origin xyz="0 0 0.05" rpy="0 0 0"/>
+    <geometry>
+      <box size="0.4 0.3 0.2"/>
+    </geometry>
+  </collision>
+  <visual>
+    <origin xyz="0 0 0.05" rpy="0 0 0"/>
+    <geometry>
+      <box size="0.4 0.3 0.2"/>
+    </geometry>
+    <material name="black"/>
+  </visual>
+  <inertial>
+    <origin xyz="0 0 0.05" rpy="0 0 0"/>
+    <mass value="1"/>
+    <inertia
+      ixx="0.01" ixy="0.0" ixz="0.0"
+      iyy="0.01" iyz="0.0"
+      izz="0.01"/>
+  </inertial>
+  </link>
+  <!-- Link Roue -->
+  <!-- link Roue Folle -->
+  <link name="RoueF">
+  <collision>
+    <origin xyz="0 0 0" rpy="0 0 0"/>
+    <geometry>
+      <sphere radius="0.05"/>
+    </geometry>
+  </collision>
+  <visual>
+    <origin xyz="0 0 0" rpy="0 0 0"/>
+    <geometry>
+      <sphere radius="0.05"/>
+    </geometry>
+    <material name="black"/>
+  </visual>
+  <inertial>
+    <origin xyz="0 0 0" rpy="0 0 0"/>
+    <mass value="0.01"/>
+    <inertia
+      ixx="0.01" ixy="0.0" ixz="0.0"
+      iyy="0.01" iyz="0.0"
+      izz="0.01"/>
+  </inertial>
+  </link>
+  <!-- link Roue Gauche -->
+  <link name="RoueG">
+  <collision>
+    <origin xyz="0 0 0" rpy="0 1.5707 1.5707"/>
+    <geometry>
+      <cylinder radius="0.15" length="0.1"/>
+    </geometry>
+  </collision>
+  <visual>
+    <origin xyz="0 0 0" rpy="0 1.5707 1.5707"/>
+    <geometry>
+      <cylinder radius="0.15" length="0.1"/>
+    </geometry>
+    <material name="black"/>
+  </visual>
+  <inertial>
+    <origin xyz="0 0 0" rpy="0 0 0"/>
+    <mass value="0.01"/>
+    <inertia
+      ixx="0.01" ixy="0.0" ixz="0.0"
+      iyy="0.01" iyz="0.0"
+      izz="0.01"/>
+  </inertial>
+  </link>
+  <!-- link Roue Droite -->
+  <link name="RoueD">
+  <collision>
+    <origin xyz="0 0 0" rpy="0 1.5707 1.5707"/>
+    <geometry>
+      <cylinder radius="0.15" length="0.1"/>
+    </geometry>
+  </collision>
+  <visual>
+    <origin xyz="0 0 0" rpy="0 1.5707 1.5707"/>
+    <geometry>
+      <cylinder radius="0.15" length="0.1"/>
+    </geometry>
+    <material name="black"/>
+  </visual>
+  <inertial>
+    <origin xyz="0 0 0" rpy="0 0 0"/>
+    <mass value="0.01"/>
+    <inertia
+      ixx="0.01" ixy="0.0" ixz="0.0"
+      iyy="0.01" iyz="0.0"
+      izz="0.01"/>
+  </inertial>
+  </link>
+  <!-- link Mat -->
+  <link name="Mat">
+  <collision>
+    <origin xyz="0 0 0" rpy="0 0 0"/>
+    <geometry>
+      <cylinder radius="0.01" length="0.2"/>
+    </geometry>
+  </collision>
+  <visual>
+    <origin xyz="0 0 0" rpy="0 0 0"/>
+    <geometry>
+      <cylinder radius="0.01" length="0.2"/>
+    </geometry>
+    <material name="black"/>
+  </visual>
+  <inertial>
+    <origin xyz="0 0 0" rpy="0 0 0"/>
+    <mass value="0.01"/>
+    <inertia
+      ixx="0.01" ixy="0.0" ixz="0.0"
+      iyy="0.01" iyz="0.0"
+      izz="0.01"/>
+  </inertial>
+  </link>
+  <!-- link Bras -->
+  <!-- link Bras Cylindre 1 -->
+  <link name="BrasC1">
+  <collision>
+    <origin xyz="0 0 0" rpy="0 0 0"/>
+    <geometry>
+      <cylinder radius="0.01" length="0.25"/>
+    </geometry>
+  </collision>
+  <visual>
+    <origin xyz="0 0 0" rpy="0 0 0"/>
+    <geometry>
+      <cylinder radius="0.01" length="0.25"/>
+    </geometry>
+    <material name="black"/>
+  </visual>
+  <inertial>
+    <origin xyz="0 0 0" rpy="0 0 0"/>
+    <mass value="0.01"/>
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
File: desherborator_description/urdf/desherborator.parameters.xacro (robot description, xacro)
@@ -1,4 +1,4 @@
 <?xml version="1.0"?>
-<robot name="desherborator_parametors" xmlns:xacro="http://www.ros.org/wiki/xacro">
+<robot name="desherborator_parameters" xmlns:xacro="http://ros.org/wiki/xacro">
     <xacro:property name="chassisHeight" value="0.2"/>
     <xacro:property name="chassisWidth" value="0.3"/>

File: desherborator_description/urdf/desherborator.sensor.xacro (robot description, xacro)
@@ -1,14 +1,4 @@
-<<<<<<< HEAD
-=======
 <?xml version="1.0"?>
-<!-- Create the robot sensors. The robot has the following sensors :
-    Lidar : an hokuyo sensor
-    Camera : Front camera of the robot
-    Laser : the laser for burning the weeds
-    Author : Elodie NOELE -->
 <robot name="desherborator_sensor" xmlns:xacro="http://ros.org/wiki/xacro">
-    <xacro:include filename="./desherborator.parameters.xacro" />
-    <xacro:include filename="./desherborator.materials.xacro" />
-    <xacro:include filename="./desherborator.joint.xacro" />
     <xacro:property name="chassisHeight" value="0.1"/>
     <xacro:macro name="LIDAR">
@@ -177,3 +167,2 @@
     </xacro:macro>
 </robot>
->>>>>>> ebd1b56c8572ec700446aef171f7176dea457216

File: desherborator_description/urdf/desherborator.urdf.xacro (robot description, xacro)
@@ -2,7 +2,8 @@
 <robot name="desherborator" xmlns:xacro="http://ros.org/wiki/xacro">
   <xacro:include filename="$(find desherborator_description)/urdf/desherborator.joint.xacro"/>
-  <!--<xacro:include filename="$(find desherborator_description)/urdf/desherborator.link.xacro"/>
+  <xacro:include filename="$(find desherborator_description)/urdf/desherborator.link.xacro"/>
   <xacro:include filename="$(find desherborator_description)/urdf/desherborator.materials.xacro"/>
-  <xacro:include filename="$(find desherborator_description)/urdf/desherborator.sensor.xacro"/>
+    <xacro:include filename="$(find desherborator_description)/urdf/desherborator.parameters.xacro"/>
+  <!--<xacro:include filename="$(find desherborator_description)/urdf/desherborator.sensor.xacro"/>
     -->
 </robot>
