Commit message: Task 1.5 & Task 1.6 : Fix robot joints and show the materials

File: desherborator_description/urdf/desherborator.joint.xacro (robot description, xacro)
@@ -30,10 +30,10 @@
         <joint name="joint_4" type="continuous">
                 <parent link="Chassis"/>
-                <child link="BrasC1"/>
+                <child link="BrasC1dummy"/>
                 <origin xyz="0.01 -0.15 0" rpy="0 0 0"/>
                 <axis  xyz="0 0 1"/>
         </joint>
         <joint name="joint_5" type="prismatic">
-                <parent link="Chassis"/>
+                <parent link="BrasC1dummy"/>
                 <child link="BrasC1"/>
                 <origin xyz="0 0 0.01" rpy="0 0 0"/>

File: desherborator_description/urdf/desherborator.link.xacro (robot description, xacro)
@@ -16,5 +16,4 @@
       <box size="0.4 0.3 0.2"/>
     </geometry>
-    <material name="black"/>
   </visual>
   <inertial>
@@ -41,5 +40,4 @@
       <sphere radius="0.05"/>
     </geometry>
-    <material name="black"/>
   </visual>
   <inertial>
@@ -65,5 +63,4 @@
       <cylinder radius="0.15" length="0.1"/>
     </geometry>
-    <material name="black"/>
   </visual>
   <inertial>
@@ -89,5 +86,4 @@
       <cylinder radius="0.15" length="0.1"/>
     </geometry>
-    <material name="black"/>
   </visual>
   <inertial>
@@ -113,5 +109,4 @@
       <cylinder radius="0.01" length="0.2"/>
     </geometry>
-    <material name="black"/>
   </visual>
   <inertial>
@@ -138,15 +133,16 @@
       <cylinder radius="0.01" length="0.25"/>
     </geometry>
-    <material name="black"/>
-  </visual>
-  <inertial>
-    <origin xyz="0 0 0" rpy="0 0 0"/>
-    <mass value="0.01"/>
-    <inertia
-      ixx="0.01" ixy="0.0" ixz="0.0"
-      iyy="0.01" iyz="0.0"
-      izz="0.01"/>
-  </inertial>
-  </link>
+  </visual>
+  <inertial>
+    <origin xyz="0 0 0" rpy="0 0 0"/>
+    <mass value="0.01"/>
+    <inertia
+      ixx="0.01" ixy="0.0" ixz="0.0"
+      iyy="0.01" iyz="0.0"
+      izz="0.01"/>
+  </inertial>
+  </link>
+  <!-- link Dummy Bras Cylindre 1 -->
+  <link name="BrasC1dummy"/>
   <!-- link Bras Cylindre 2 -->
   <link name="BrasC2">
@@ -162,5 +158,4 @@
       <cylinder radius="0.01" length="0.3"/>
     </geometry>
-    <material name="black"/>
   </visual>
   <inertial>
@@ -186,5 +181,4 @@
       <cylinder radius="0.01" length="0.1"/>
     </geometry>
-    <material name="black"/>
   </visual>
   <inertial>
@@ -210,5 +204,4 @@
       <sphere radius="0.02"/>
     </geometry>
-    <material name="black"/>
   </visual>
   <inertial>
@@ -234,5 +227,4 @@
       <sphere radius="0.02"/>
     </geometry>
-    <material name="black"/>
   </visual>
   <inertial>

File: desherborator_description/urdf/desherborator.materials.xacro (robot description, xacro)
@@ -3,27 +3,51 @@
     Author : Elodie NOELE -->
 <robot name="desherborator_materials" xmlns:xacro="http://ros.org/wiki/xacro">
-  <material name="black">
-    <color rgba="0.0 0.0 0.0 1.0"/>
-  </material>
-  <material name="blue">
-    <color rgba="0.0 0.0 0.8 1.0"/>
-  </material>
-  <material name="green">
-    <color rgba="0.0 0.8 0.0 1.0"/>
-  </material>
-  <material name="gray">
-    <color rgba="0.7 0.7 0.7 1.0"/>
-  </material>
-  <material name="darkgray">
-    <color rgba="0.3 0.3 0.3 1.0"/>
-  </material>
-  <material name="red">
-    <color rgba="0.8 0.0 0.0 1.0"/>
-  </material>
-  <material name="white">
-    <color rgba="1.0 1.0 1.0 1.0"/>
-  </material>
-  <material name="yellow">
-    <color rgba="0.8 0.8 0.0 1.0"/>
-  </material>
+  <gazebo reference="Chassis">
+    <material>Gazebo/DarkGrey</material>
+  </gazebo>
+  <gazebo reference="RoueG">
+    <mu1>1.2</mu1>
+    <mu2>1.2</mu2>
+    <kp>500000.0</kp>
+    <kd>10.0</kd>
+    <minDepth>0.001</minDepth>
+    <maxVel>0.1</maxVel>
+    <material>Gazebo/FlatBlack</material>
+  </gazebo>
+  <gazebo reference="RoueD">
+    <mu1>1.2</mu1>
+    <mu2>1.2</mu2>
+    <kp>500000.0</kp>
+    <kd>10.0</kd>
+    <minDepth>0.001</minDepth>
+    <maxVel>0.1</maxVel>
+    <material>Gazebo/FlatBlack</material>
+  </gazebo>
+  <gazebo reference="RoueF">
+    <mu1>0.1</mu1>
+    <mu2>0.1</mu2>
+    <kp>1000000.0</kp>
+    <kd>100.0</kd>
+    <minDepth>0.001</minDepth>
+    <maxVel>1.0</maxVel>
+    <material>Gazebo/FlatBlack</material>
+  </gazebo>
+  <gazebo reference="Mat">
+    <material>Gazebo/FlatBlack</material>
+  </gazebo>
+  <gazebo reference="BrasC1">
+    <material>Gazebo/FlatBlack</material>
+  </gazebo>
+  <gazebo reference="BrasC2">
+    <material>Gazebo/FlatBlack</material>
+  </gazebo>
+  <gazebo reference="BrasC3">
+    <material>Gazebo/FlatBlack</material>
+  </gazebo>
+  <gazebo reference="BrasS1">
+    <material>Gazebo/FlatBlack</material>
+  </gazebo>
+  <gazebo reference="BrasS2">
+    <material>Gazebo/FlatBlack</material>
+  </gazebo>
 </robot>

File: desherborator_description/urdf/desherborator.sensor.xacro (robot description, xacro)
@@ -3,5 +3,5 @@
     <xacro:macro name="LIDAR">
         <gazebo reference="LIDAR">
-            <material name= "black"/>
+            <material>Gazebo/Black</material>
             <sensor type="ray" name="lidar_sensor">
             <pose>0 0 0 0 0 0</pose>
@@ -52,43 +52,43 @@
     <xacro:macro name="Camera">
         <gazebo reference="Camera">
-            <material name= "red"/>
+            <material>Gazebo/Red</material>
             <sensor type="camera" name="main_camera">
-            <update_rate>30.0</update_rate>
-            <camera name="head">
-                <horizontal_fov>1.3962634</horizontal_fov>
-                <image>
-                <width>1280</width>
-                <height>720</height>
-                <format>R8G8B8</format>
-                </image>
-                <clip>
-                <near>0.02</near>
-                <far>300</far>
-                </clip>
-                <noise>
-                <type>gaussian</type>
-                <mean>0.0</mean>
-                <stddev>0.007</stddev>
-                </noise>
-            </camera>
-            <plugin name="camera_controller" filename="libgazebo_ros_camera.so">
-                <alwaysOn>true</alwaysOn>
-                <updateRate>0.0</updateRate>
-                <cameraName>main_camera</cameraName>
-                <imageTopicName>image_raw</imageTopicName>
-                <cameraInfoTopicName>camera_info</cameraInfoTopicName>
-                <frameName>camera</frameName>
-                <hackBaseline>0.07</hackBaseline>
-                <distortionK1>0.0</distortionK1>
-                <distortionK2>0.0</distortionK2>
-                <distortionK3>0.0</distortionK3>
-                <distortionT1>0.0</distortionT1>
-                <distortionT2>0.0</distortionT2>
-            </plugin>
+                <update_rate>30.0</update_rate>
+                <camera name="head">
+                    <horizontal_fov>1.3962634</horizontal_fov>
+                    <image>
+                    <width>1280</width>
+                    <height>720</height>
+                    <format>R8G8B8</format>
+                    </image>
+                    <clip>
+                    <near>0.02</near>
+                    <far>300</far>
+                    </clip>
+                    <noise>
+                    <type>gaussian</type>
+                    <mean>0.0</mean>
+                    <stddev>0.007</stddev>
+                    </noise>
+                </camera>
+                <plugin name="camera_controller" filename="libgazebo_ros_camera.so">
+                    <alwaysOn>true</alwaysOn>
+                    <updateRate>0.0</updateRate>
+                    <cameraName>main_camera</cameraName>
+                    <imageTopicName>image_raw</imageTopicName>
+                    <cameraInfoTopicName>camera_info</cameraInfoTopicName>
+                    <frameName>camera</frameName>
+                    <hackBaseline>0.07</hackBaseline>
+                    <distortionK1>0.0</distortionK1>
+                    <distortionK2>0.0</distortionK2>
+                    <distortionK3>0.0</distortionK3>
+                    <distortionT1>0.0</distortionT1>
+                    <distortionT2>0.0</distortionT2>
+                </plugin>
             </sensor>
         </gazebo>
         <joint name="camera_joint" type="fixed">
             <parent link="chassis"/>
-            <axis xyz="0 1 0" />
+            <axis xyz="10 10 10" />
             <origin xyz="${chassisWidth} 0 ${chassisHeight/2}" rpy="0 0 0"/>
             <child link="camera_link"/>
@@ -118,5 +118,5 @@
     <xacro:macro name="LASER">
         <gazebo reference="LASER">
-            <material name= "blue"/>
+            <material>Gazebo/Blue</material>
             <sensor type="ray" name="laser_sensor">
             <pose>0 0 0 0 0 0</pose>

File: desherborator_description/urdf/desherborator.urdf (robot description, URDF)
Before this commit: robot desherborator, 11 links, 11 joints
Links:
- added link BrasC1dummy
Joints:
- joint joint_4: child BrasC1 -> BrasC1dummy
- joint joint_5: parent Chassis -> BrasC1dummy

File: desherborator_description/urdf/desherborator.urdf.xacro (robot description, xacro)
@@ -1,8 +1,33 @@
 <?xml version="1.0"?>
 <robot name="desherborator" xmlns:xacro="http://ros.org/wiki/xacro">
-  <xacro:include filename="$(find desherborator_description)/urdf/desherborator.joint.xacro"/>
-  <xacro:include filename="$(find desherborator_description)/urdf/desherborator.link.xacro"/>
-  <xacro:include filename="$(find desherborator_description)/urdf/desherborator.sensor.xacro"/>
   <xacro:include filename="$(find desherborator_description)/urdf/desherborator.materials.xacro"/>
   <xacro:include filename="$(find desherborator_description)/urdf/desherborator.parameters.xacro"/>
+  <xacro:include filename="$(find desherborator_description)/urdf/desherborator.link.xacro"/>
+  <xacro:include filename="$(find desherborator_description)/urdf/desherborator.joint.xacro"/>
+  <xacro:include filename="$(find desherborator_description)/urdf/desherborator.sensor.xacro"/>
+  <gazebo>
+    <plugin name="wheels_controller" filename="libgazebo_ros_diff_drive.so">
+      <commandTopic>cmd_vel</commandTopic>
+      <odometryTopic>odom</odometryTopic>
+      <odometryFrame>odom</odometryFrame>
+      <odometrySource>world</odometrySource>
+      <publishOdomTF>true</publishOdomTF>
+      <!-- ENTER BASE LINK NAME -->
+      <robotBaseFrame>base_link</robotBaseFrame>
+      <publishWheelTF>true</publishWheelTF>
+      <publishTf>true</publishTf>
+      <publishWheelJointState>true</publishWheelJointState>
+      <legacyMode>true</legacyMode>
+      <updateRate>30</updateRate>
+      <!-- ENTER LEFT JOINT NAME -->
+      <leftJoint>RoueG</leftJoint>
+      <!-- ENTER RIGHT JOINT NAME -->
+      <rightJoint>RoueD</rightJoint>
+      <wheelSeparation>0.31</wheelSeparation>
+      <wheelDiameter>0.1</wheelDiameter>
+      <wheelAcceleration>0.1</wheelAcceleration>
+      <wheelTorque>10</wheelTorque>
+      <rosDebugLevel>na</rosDebugLevel>
+    </plugin>
+  </gazebo>
 </robot>

Commit message: Task 1.3 : Create robot sensors (not finished)

File: desherborator_description/urdf/desherborator.joint.xacro (robot description, xacro)
@@ -1,4 +1,4 @@
 <?xml version="1.0"?>
-<robot name="desherborator_joints" xmlns:xacro="http://ros.org/wiki/xacro">
+<robot name="desherborator" xmlns:xacro="http://ros.org/wiki/xacro">
         <joint name="base_joint" type="fixed">
                 <parent link="base_link"/>

File: desherborator_description/urdf/desherborator.link.xacro (robot description, xacro)
@@ -1,121 +1,121 @@
 <?xml version="1.0"?>
-<robot name="desherborator_links" xmlns:xacro="http://ros.org/wiki/xacro">
+<robot name="desherborator" xmlns:xacro="http://ros.org/wiki/xacro">
   <!-- Base Chassis -->
   <link name="base_link"/>
   <!-- Link Chassis -->
   <link name="Chassis">
-  <collision>
-    <origin xyz="0 0 0.05" rpy="0 0 0"/>
-    <geometry>
-      <box size="0.4 0.3 0.2"/>
-    </geometry>
-  </collision>
-  <visual>
-    <origin xyz="0 0 0.05" rpy="0 0 0"/>
-    <geometry>
-      <box size="0.4 0.3 0.2"/>
-    </geometry>
-  </visual>
-  <inertial>
-    <origin xyz="0 0 0.05" rpy="0 0 0"/>
-    <mass value="1"/>
-    <inertia
-      ixx="0.01" ixy="0.0" ixz="0.0"
-      iyy="0.01" iyz="0.0"
-      izz="0.01"/>
-  </inertial>
+    <collision>
+      <origin xyz="0 0 0.05" rpy="0 0 0"/>
+      <geometry>
+        <box size="0.4 0.3 0.2"/>
+      </geometry>
+    </collision>
+    <visual>
+      <origin xyz="0 0 0.05" rpy="0 0 0"/>
+      <geometry>
+        <box size="0.4 0.3 0.2"/>
+      </geometry>
+    </visual>
+    <inertial>
+      <origin xyz="0 0 0.05" rpy="0 0 0"/>
+      <mass value="1"/>
+      <inertia
+        ixx="0.01" ixy="0.0" ixz="0.0"
+        iyy="0.01" iyz="0.0"
+        izz="0.01"/>
+    </inertial>
   </link>
   <!-- Link Roue -->
   <!-- link Roue Folle -->
   <link name="RoueF">
-  <collision>
-    <origin xyz="0 0 0" rpy="0 0 0"/>
-    <geometry>
-      <sphere radius="0.05"/>
-    </geometry>
-  </collision>
-  <visual>
-    <origin xyz="0 0 0" rpy="0 0 0"/>
-    <geometry>
-      <sphere radius="0.05"/>
-    </geometry>
-  </visual>
-  <inertial>
-    <origin xyz="0 0 0" rpy="0 0 0"/>
-    <mass value="0.01"/>
-    <inertia
-      ixx="0.01" ixy="0.0" ixz="0.0"
-      iyy="0.01" iyz="0.0"
-      izz="0.01"/>
-  </inertial>
+    <collision>
+      <origin xyz="0 0 0" rpy="0 0 0"/>
+      <geometry>
+        <sphere radius="0.05"/>
+      </geometry>
+    </collision>
+    <visual>
+      <origin xyz="0 0 0" rpy="0 0 0"/>
+      <geometry>
+        <sphere radius="0.05"/>
+      </geometry>
+    </visual>
+    <inertial>
+      <origin xyz="0 0 0" rpy="0 0 0"/>
+      <mass value="0.01"/>
+      <inertia
+        ixx="0.01" ixy="0.0" ixz="0.0"
+        iyy="0.01" iyz="0.0"
+        izz="0.01"/>
+    </inertial>
   </link>
   <!-- link Roue Gauche -->
   <link name="RoueG">
-  <collision>
-    <origin xyz="0 0 0" rpy="0 1.5707 1.5707"/>
-    <geometry>
-      <cylinder radius="0.15" length="0.1"/>
-    </geometry>
-  </collision>
-  <visual>
-    <origin xyz="0 0 0" rpy="0 1.5707 1.5707"/>
-    <geometry>
-      <cylinder radius="0.15" length="0.1"/>
-    </geometry>
-  </visual>
-  <inertial>
-    <origin xyz="0 0 0" rpy="0 0 0"/>
-    <mass value="0.01"/>
-    <inertia
-      ixx="0.01" ixy="0.0" ixz="0.0"
-      iyy="0.01" iyz="0.0"
-      izz="0.01"/>
-  </inertial>
+    <collision>
+      <origin xyz="0 0 0" rpy="0 1.5707 1.5707"/>
+      <geometry>
+        <cylinder radius="0.15" length="0.1"/>
+      </geometry>
+    </collision>
+    <visual>
+      <origin xyz="0 0 0" rpy="0 1.5707 1.5707"/>
+      <geometry>
+        <cylinder radius="0.15" length="0.1"/>
+      </geometry>
+    </visual>
+    <inertial>
+      <origin xyz="0 0 0" rpy="0 0 0"/>
+      <mass value="0.01"/>
+      <inertia
+        ixx="0.01" ixy="0.0" ixz="0.0"
+        iyy="0.01" iyz="0.0"
+        izz="0.01"/>
+    </inertial>
   </link>
   <!-- link Roue Droite -->
   <link name="RoueD">
-  <collision>
-    <origin xyz="0 0 0" rpy="0 1.5707 1.5707"/>
-    <geometry>
-      <cylinder radius="0.15" length="0.1"/>
-    </geometry>
-  </collision>
-  <visual>
-    <origin xyz="0 0 0" rpy="0 1.5707 1.5707"/>
-    <geometry>
-      <cylinder radius="0.15" length="0.1"/>
-    </geometry>
-  </visual>
-  <inertial>
-    <origin xyz="0 0 0" rpy="0 0 0"/>
-    <mass value="0.01"/>
-    <inertia
-      ixx="0.01" ixy="0.0" ixz="0.0"
-      iyy="0.01" iyz="0.0"
-      izz="0.01"/>
-  </inertial>
+    <collision>
+      <origin xyz="0 0 0" rpy="0 1.5707 1.5707"/>
+      <geometry>
+        <cylinder radius="0.15" length="0.1"/>
+      </geometry>
+    </collision>
+    <visual>
+      <origin xyz="0 0 0" rpy="0 1.5707 1.5707"/>
+      <geometry>
+        <cylinder radius="0.15" length="0.1"/>
+      </geometry>
+    </visual>
+    <inertial>
+      <origin xyz="0 0 0" rpy="0 0 0"/>
+      <mass value="0.01"/>
+      <inertia
+        ixx="0.01" ixy="0.0" ixz="0.0"
+        iyy="0.01" iyz="0.0"
+        izz="0.01"/>
+    </inertial>
   </link>
   <!-- link Mat -->
   <link name="Mat">
-  <collision>
-    <origin xyz="0 0 0" rpy="0 0 0"/>
-    <geometry>
-      <cylinder radius="0.01" length="0.2"/>
-    </geometry>
-  </collision>
-  <visual>
-    <origin xyz="0 0 0" rpy="0 0 0"/>
-    <geometry>
-      <cylinder radius="0.01" length="0.2"/>
-    </geometry>
-  </visual>
-  <inertial>
-    <origin xyz="0 0 0" rpy="0 0 0"/>
-    <mass value="0.01"/>
-    <inertia
-      ixx="0.01" ixy="0.0" ixz="0.0"
-      iyy="0.01" iyz="0.0"
-      izz="0.01"/>
-  </inertial>
+    <collision>
+      <origin xyz="0 0 0" rpy="0 0 0"/>
+      <geometry>
+        <cylinder radius="0.01" length="0.2"/>
+      </geometry>
+    </collision>
+    <visual>
+      <origin xyz="0 0 0" rpy="0 0 0"/>
+      <geometry>
+        <cylinder radius="0.01" length="0.2"/>
+      </geometry>
+    </visual>
+    <inertial>
+      <origin xyz="0 0 0" rpy="0 0 0"/>
+      <mass value="0.01"/>
+      <inertia
+        ixx="0.01" ixy="0.0" ixz="0.0"
+        iyy="0.01" iyz="0.0"
+        izz="0.01"/>
+    </inertial>
   </link>
   <!-- link Bras -->
@@ -147,93 +147,93 @@
   <!-- link Bras Cylindre 2 -->
   <link name="BrasC2">
-  <collision>
-    <origin xyz="0 0 0" rpy="0 1.5707 1.5707"/>
-    <geometry>
-      <cylinder radius="0.01" length="0.3"/>
-    </geometry>
-  </collision>
-  <visual>
-    <origin xyz="0 0 0" rpy="0 0 0"/>
-    <geometry>
-      <cylinder radius="0.01" length="0.3"/>
-    </geometry>
-  </visual>
-  <inertial>
-    <origin xyz="0 0 0" rpy="0 1.5707 1.5707"/>
-    <mass value="0.01"/>
-    <inertia
-      ixx="0.01" ixy="0.0" ixz="0.0"
-      iyy="0.01" iyz="0.0"
-      izz="0.01"/>
-  </inertial>
+    <collision>
+      <origin xyz="0 0 0" rpy="0 1.5707 1.5707"/>
+      <geometry>
+        <cylinder radius="0.01" length="0.3"/>
+      </geometry>
+    </collision>
+    <visual>
+      <origin xyz="0 0 0" rpy="0 0 0"/>
+      <geometry>
+        <cylinder radius="0.01" length="0.3"/>
+      </geometry>
+    </visual>
+    <inertial>
+      <origin xyz="0 0 0" rpy="0 1.5707 1.5707"/>
+      <mass value="0.01"/>
+      <inertia
+        ixx="0.01" ixy="0.0" ixz="0.0"
+        iyy="0.01" iyz="0.0"
+        izz="0.01"/>
+    </inertial>
   </link>
   <!-- link Bras Cylindre 3 -->
   <link name="BrasC3">
-  <collision>
-    <origin xyz="0 0 0" rpy="0 3.14 0"/>
-    <geometry>
-      <cylinder radius="0.01" length="0.1"/>
-    </geometry>
-  </collision>
-  <visual>
-    <origin xyz="0 0 0" rpy="0 3.14 0"/>
-    <geometry>
-      <cylinder radius="0.01" length="0.1"/>
-    </geometry>
-  </visual>
-  <inertial>
-    <origin xyz="0 0 0" rpy="0 0 0"/>
-    <mass value="0.01"/>
-    <inertia
-      ixx="0.01" ixy="0.0" ixz="0.0"
-      iyy="0.01" iyz="0.0"
-      izz="0.01"/>
-  </inertial>
+    <collision>
+      <origin xyz="0 0 0" rpy="0 3.14 0"/>
+      <geometry>
+        <cylinder radius="0.01" length="0.1"/>
+      </geometry>
+    </collision>
+    <visual>
+      <origin xyz="0 0 0" rpy="0 3.14 0"/>
+      <geometry>
+        <cylinder radius="0.01" length="0.1"/>
+      </geometry>
+    </visual>
+    <inertial>
+      <origin xyz="0 0 0" rpy="0 0 0"/>
+      <mass value="0.01"/>
+      <inertia
+        ixx="0.01" ixy="0.0" ixz="0.0"
+        iyy="0.01" iyz="0.0"
+        izz="0.01"/>
+    </inertial>
   </link>
   <!-- link Bras Sphere 1 -->
   <link name="BrasS1">
-  <collision>
-    <origin xyz="0 0 0" rpy="0 0 0"/>
-    <geometry>
-      <sphere radius="0.02"/>
-    </geometry>
-  </collision>
-  <visual>
-    <origin xyz="0 0 0" rpy="0 0 0"/>
-    <geometry>
-      <sphere radius="0.02"/>
-    </geometry>
-  </visual>
-  <inertial>
-    <origin xyz="0 0 0" rpy="0 0 0"/>
-    <mass value="0.01"/>
-    <inertia
-      ixx="0.01" ixy="0.0" ixz="0.0"
-      iyy="0.01" iyz="0.0"
-      izz="0.01"/>
-  </inertial>
+    <collision>
+      <origin xyz="0 0 0" rpy="0 0 0"/>
+      <geometry>
+        <sphere radius="0.02"/>
+      </geometry>
+    </collision>
+    <visual>
+      <origin xyz="0 0 0" rpy="0 0 0"/>
+      <geometry>
+        <sphere radius="0.02"/>
+      </geometry>
+    </visual>
+    <inertial>
+      <origin xyz="0 0 0" rpy="0 0 0"/>
+      <mass value="0.01"/>
+      <inertia
+        ixx="0.01" ixy="0.0" ixz="0.0"
+        iyy="0.01" iyz="0.0"
+        izz="0.01"/>
+    </inertial>
   </link>
   <!-- link Bras Sphere 2 -->
   <link name="BrasS2">
-  <collision>
-    <origin xyz="0 0 0" rpy="0 0 0"/>
-    <geometry>
-      <sphere radius="0.02"/>
-    </geometry>
-  </collision>
-  <visual>
-    <origin xyz="0 0 0" rpy="0 0 0"/>
-    <geometry>
-      <sphere radius="0.02"/>
-    </geometry>
-  </visual>
-  <inertial>
-    <origin xyz="0 0 0" rpy="0 0 0"/>
-    <mass value="0.01"/>
-    <inertia
-      ixx="0.01" ixy="0.0" ixz="0.0"
-      iyy="0.01" iyz="0.0"
-      izz="0.01"/>
-  </inertial>
+    <collision>
+      <origin xyz="0 0 0" rpy="0 0 0"/>
+      <geometry>
+        <sphere radius="0.02"/>
+      </geometry>
+    </collision>
+    <visual>
+      <origin xyz="0 0 0" rpy="0 0 0"/>
+      <geometry>
+        <sphere radius="0.02"/>
+      </geometry>
+    </visual>
+    <inertial>
+      <origin xyz="0 0 0" rpy="0 0 0"/>
+      <mass value="0.01"/>
+      <inertia
+        ixx="0.01" ixy="0.0" ixz="0.0"
+        iyy="0.01" iyz="0.0"
+        izz="0.01"/>
+    </inertial>
   </link>
 </robot>

File: desherborator_description/urdf/desherborator.materials.xacro (robot description, xacro)
@@ -2,5 +2,5 @@
 <!-- Here are defined the materials used for defining the robot in the simulation
     Author : Elodie NOELE -->
-<robot name="desherborator_materials" xmlns:xacro="http://ros.org/wiki/xacro">
+<robot name="desherborator" xmlns:xacro="http://ros.org/wiki/xacro">
   <gazebo reference="Chassis">
     <material>Gazebo/DarkGrey</material>

File: desherborator_description/urdf/desherborator.parameters.xacro (robot description, xacro)
@@ -1,10 +1,14 @@
 <?xml version="1.0"?>
-<robot name="desherborator_parameters" xmlns:xacro="http://ros.org/wiki/xacro">
-    <xacro:property name="chassisHeight" value="0.2"/>
-    <xacro:property name="chassisWidth" value="0.3"/>
+<robot name="desherborator" xmlns:xacro="http://ros.org/wiki/xacro">
+    <xacro:property name="ChassisHeight" value="0.2"/>
+    <xacro:property name="ChassisWidth" value="0.3"/>
     <xacro:property name="cameraSize" value="0.1"/>
-    <xacro:property name="lidarRadius" value="0.3"/>
-    <xacro:property name="lidarLength" value="0.4"/>
-    <xacro:property name="laserRadius" value="0.025"/>
-    <xacro:property name="laserLength" value="0.15"/>
+    <xacro:property name="wheelRadius" value="0.15"/>
+    <xacro:property name="wheelWidth" value="0.1"/>
+    <xacro:macro name="default_inertial" params="mass">
+        <inertial>
+        <mass value="${mass}" />
+        <inertia ixx="0.01" ixy="0.0" ixz="0.0" iyy="0.01" iyz="0.0" izz="0.01" />
+        </inertial>
+    </xacro:macro>
 </robot>
