Commit message: Task 1.3 : Create robot sensors (not finished)

File: desherborator_description/urdf/desherborator.sensor.xacro (robot description, xacro)
@@ -1,167 +1,163 @@
 <?xml version="1.0"?>
-<robot name="desherborator_sensor" xmlns:xacro="http://ros.org/wiki/xacro">
-    <xacro:macro name="LIDAR">
-        <gazebo reference="LIDAR">
-            <material>Gazebo/Black</material>
-            <sensor type="ray" name="lidar_sensor">
-            <pose>0 0 0 0 0 0</pose>
-            <visualize>true</visualize>
-            <update_rate>5</update_rate>
-            <ray>
-                <scan>
-                <horizontal>
-                    <samples>720</samples>
-                    <resolution>1</resolution>
-                    <min_angle>0.0</min_angle>
-                    <max_angle>6.28319</max_angle>
-                </horizontal>
-                </scan>
-                <range>
-                <min>0.120</min>
-                <max>12</max>
-                <resolution>0.015</resolution>
-                </range>
+<robot name="desherborator" xmlns:xacro="http://ros.org/wiki/xacro">
+    <link name="LIDAR">
+        <visual>
+        <origin xyz="0 0 0" rpy="0 0 0"/>
+        <geometry>
+            <cylinder radius="0.03" length="0.04"/>
+        </geometry>
+        </visual>
+        <xacro:default_inertial mass="0.1"/>
+    </link>
+    <joint name="lidar_joint" type="fixed">
+        <parent link="Chassis"/>
+        <child link="LIDAR"/>
+        <origin xyz="0.15 0 0.23" rpy="0 0 0"/>
+    </joint>
+    <gazebo reference="LIDAR">
+        <material>Gazebo/Orange</material>
+        <sensor type="ray" name="lidar_sensor">
+        <pose>0 0 0 0 0 0</pose>
+        <visualize>true</visualize>
+        <update_rate>40</update_rate>
+        <ray>
+            <scan>
+            <horizontal>
+                <samples>720</samples>
+                <resolution>1</resolution>
+                <min_angle>0.0</min_angle>
+                <max_angle>6.28319</max_angle>
+            </horizontal>
+            </scan>
+            <range>
+            <min>0.120</min>
+            <max>12</max>
+            <resolution>0.015</resolution>
+            </range>
+            <noise>
+            <type>gaussian</type>
+            <mean>0.0</mean>
+            <stddev>0.01</stddev>
+            </noise>
+        </ray>
+        <plugin name="gazebo_ros_lds_lfcd_controller" filename="libgazebo_ros_laser.so">
+            <topicName>scan</topicName>
+            <!-- ENTER FRAME NAME -->
+            <frameName>LIDAR</frameName>
+        </plugin>
+        </sensor>
+    </gazebo>
+    <joint name="camera_joint" type="fixed">
+        <parent link="Chassis"/>
+        <axis xyz="0 0 0" />
+        <origin xyz="${ChassisWidth} 0 ${ChassisHeight/2}" rpy="0 0 0"/>
+        <child link="Camera"/>
+    </joint>
+    <!-- Camera -->
+    <link name="Camera">
+        <collision>
+        <origin xyz="0 0 0" rpy="0 0 0"/>
+        <geometry>
+        <box size="${cameraSize} ${cameraSize} ${cameraSize}"/>
+        </geometry>
+        </collision>
+        <visual>
+        <origin xyz="0 0 0" rpy="0 0 0"/>
+        <geometry>
+        <box size="${cameraSize} ${cameraSize} ${cameraSize}"/>
+        </geometry>
+        <material name="red"/>
+        </visual>
+        <inertial>
+        <mass value="1e-5" />
+        <origin xyz="0 0 0" rpy="0 0 0"/>
+        <inertia ixx="1e-6" ixy="0" ixz="0" iyy="1e-6" iyz="0" izz="1e-6" />
+        </inertial>
+    </link>
+    <gazebo reference="Camera">
+        <material>Gazebo/Green</material>
+        <sensor type="camera" name="main_camera">
+            <update_rate>30.0</update_rate>
+            <camera name="head">
+                <horizontal_fov>1.3962634</horizontal_fov>
+                <image>
+                <width>1280</width>
+                <height>720</height>
+                <format>R8G8B8</format>
+                </image>
+                <clip>
+                <near>0.02</near>
+                <far>300</far>
+                </clip>
                 <noise>
                 <type>gaussian</type>
                 <mean>0.0</mean>
-                <stddev>0.01</stddev>
+                <stddev>0.007</stddev>
                 </noise>
-            </ray>
-            <plugin name="gazebo_ros_lds_lfcd_controller" filename="libgazebo_ros_laser.so">
-                <topicName>scan</topicName>
-                <!-- ENTER FRAME NAME -->
-                <frameName>lidar</frameName>
+            </camera>
+            <plugin name="camera_controller" filename="libgazebo_ros_camera.so">
+                <topicName>camera</topicName>
+                <frameName>Camera</frameName>
+                <alwaysOn>true</alwaysOn>
+                <updateRate>0.0</updateRate>
+                <cameraName>main_camera</cameraName>
+                <imageTopicName>image_raw</imageTopicName>
+                <cameraInfoTopicName>camera_info</cameraInfoTopicName>
+                <frameName>camera</frameName>
+                <hackBaseline>0.07</hackBaseline>
+                <distortionK1>0.0</distortionK1>
+                <distortionK2>0.0</distortionK2>
+                <distortionK3>0.0</distortionK3>
+                <distortionT1>0.0</distortionT1>
+                <distortionT2>0.0</distortionT2>
             </plugin>
-            </sensor>
-        </gazebo>
-        <link name="lidar">
-            <visual>
-            <origin xyz="0 0 -0.03" rpy="0 0 0"/>
-            <geometry>
-                <cylinder radius="{lidarRadius}" length="{lidarLength}"/>
-            </geometry>
-            </visual>
-            <xacro:default_inertial mass="0.1"/>
-        </link>
-        <joint name="lidar_joint" type="fixed">
-            <parent link="chassis"/>
-            <child link="lidar"/>
-            <origin xyz="0.15 0 0.23" rpy="0 0 0"/>
-        </joint>
-    </xacro:macro>
-    <xacro:macro name="Camera">
-        <gazebo reference="Camera">
-            <material>Gazebo/Red</material>
-            <sensor type="camera" name="main_camera">
-                <update_rate>30.0</update_rate>
-                <camera name="head">
-                    <horizontal_fov>1.3962634</horizontal_fov>
-                    <image>
-                    <width>1280</width>
-                    <height>720</height>
-                    <format>R8G8B8</format>
-                    </image>
-                    <clip>
-                    <near>0.02</near>
-                    <far>300</far>
-                    </clip>
-                    <noise>
-                    <type>gaussian</type>
-                    <mean>0.0</mean>
-                    <stddev>0.007</stddev>
-                    </noise>
-                </camera>
-                <plugin name="camera_controller" filename="libgazebo_ros_camera.so">
-                    <alwaysOn>true</alwaysOn>
-                    <updateRate>0.0</updateRate>
-                    <cameraName>main_camera</cameraName>
-                    <imageTopicName>image_raw</imageTopicName>
-                    <cameraInfoTopicName>camera_info</cameraInfoTopicName>
-                    <frameName>camera</frameName>
-                    <hackBaseline>0.07</hackBaseline>
-                    <distortionK1>0.0</distortionK1>
-                    <distortionK2>0.0</distortionK2>
-                    <distortionK3>0.0</distortionK3>
-                    <distortionT1>0.0</distortionT1>
-                    <distortionT2>0.0</distortionT2>
-                </plugin>
-            </sensor>
-        </gazebo>
-        <joint name="camera_joint" type="fixed">
-            <parent link="chassis"/>
-            <axis xyz="10 10 10" />
-            <origin xyz="${chassisWidth} 0 ${chassisHeight/2}" rpy="0 0 0"/>
-            <child link="camera_link"/>
-        </joint>
-        <!-- Camera -->
-        <link name="camera_link">
-            <collision>
-            <origin xyz="0 0 0" rpy="0 0 0"/>
-            <geometry>
-            <box size="${cameraSize} ${cameraSize} ${cameraSize}"/>
-            </geometry>
-            </collision>
-            <visual>
-            <origin xyz="0 0 0" rpy="0 0 0"/>
-            <geometry>
-            <box size="${cameraSize} ${cameraSize} ${cameraSize}"/>
-            </geometry>
-            <material name="red"/>
-            </visual>
-            <inertial>
-            <mass value="1e-5" />
-            <origin xyz="0 0 0" rpy="0 0 0"/>
-            <inertia ixx="1e-6" ixy="0" ixz="0" iyy="1e-6" iyz="0" izz="1e-6" />
-            </inertial>
-        </link>
-    </xacro:macro>
-    <xacro:macro name="LASER">
-        <gazebo reference="LASER">
-            <material>Gazebo/Blue</material>
-            <sensor type="ray" name="laser_sensor">
-            <pose>0 0 0 0 0 0</pose>
-            <visualize>true</visualize>
-            <update_rate>5</update_rate>
-            <ray>
-                <scan>
-                <horizontal>
-                    <samples>720</samples>
-                    <resolution>1</resolution>
-                    <min_angle>0.0</min_angle>
-                    <max_angle>0.1</max_angle>
-                </horizontal>
-                </scan>
-                <range>
-                <min>0.120</min>
-                <max>12</max>
-                <resolution>0.015</resolution>
-                </range>
-                <noise>
-                <type>gaussian</type>
-                <mean>0.0</mean>
-                <stddev>0.01</stddev>
-                </noise>
-            </ray>
-            <plugin name="gazebo_ros_lds_lfcd_controller" filename="libgazebo_ros_laser.so">
-                <topicName>scan_laser</topicName>
-                <!-- ENTER FRAME NAME -->
-                <frameName>laser</frameName>
-            </plugin>
-            </sensor>
-        </gazebo>
-        <link name="laser">
-            <visual>
-            <origin xyz="0 0 -0.03" rpy="0 0 0"/>
-            <geometry>
-                <cylinder radius="{laserRadius}" length="{laserLength}"/>
-            </geometry>
-            </visual>
-            <xacro:default_inertial mass="0.1"/>
-        </link>
-        <joint name="laser_joint" type="fixed">
-            <parent link="chassis"/>
-            <child link="laser"/>
-            <origin xyz="0.15 0 0.23" rpy="0 0 0"/>
-        </joint>
-    </xacro:macro>
+        </sensor>
+    </gazebo>
+    <link name="LASER">
+        <visual>
+        <origin xyz="0 0 0" rpy="0 0 0"/>
+        <geometry>
+            <cylinder radius="0.025" length="0.15"/>
+        </geometry>
+        </visual>
+        <xacro:default_inertial mass="0.1"/>
+    </link>
+    <joint name="laser_joint" type="fixed">
+        <parent link="Chassis"/>
+        <child link="LASER"/>
+        <origin xyz="0.15 0 0.23" rpy="0 0 0"/>
+    </joint>
+    <gazebo reference="LASER">
+        <material>Gazebo/Blue</material>
+        <sensor type="ray" name="laser_sensor">
+        <pose>0 0 0 0 0 0</pose>
+        <visualize>true</visualize>
+        <update_rate>5</update_rate>
+        <ray>
+            <scan>
+            <horizontal>
+                <samples>720</samples>
+                <resolution>1</resolution>
+                <min_angle>0.0</min_angle>
+                <max_angle>0.1</max_angle>
+            </horizontal>
+            </scan>
+            <range>
+            <min>0.120</min>
+            <max>12</max>
+            <resolution>0.015</resolution>
+            </range>
+            <noise>
+            <type>gaussian</type>
+            <mean>0.0</mean>
+            <stddev>0.01</stddev>
+            </noise>
+        </ray>
+        <plugin name="gazebo_ros_lds_lfcd_controller" filename="libgazebo_ros_laser.so">
+            <topicName>scan_laser</topicName>
+            <!-- ENTER FRAME NAME -->
+            <frameName>laser</frameName>
+        </plugin>
+        </sensor>
+    </gazebo>
 </robot>

File: desherborator_description/urdf/desherborator.urdf (robot description, URDF)
Before this commit: robot desherborator, 12 links, 11 joints
Links:
- added link Camera, mass 1e-5; collision box size=0.1 0.1 0.1; visual box size=0.1 0.1 0.1
- added link LASER, mass 0.1; visual cylinder length=0.15 radius=0.025
- added link LIDAR, mass 0.1; visual cylinder length=0.04 radius=0.03
Joints:
- added joint camera_joint: type fixed, parent Chassis, child Camera, origin xyz=0.3 0 0.1 rpy=0 0 0, axis 0 0 0
- added joint laser_joint: type fixed, parent Chassis, child LASER, origin xyz=0.15 0 0.23 rpy=0 0 0
- added joint lidar_joint: type fixed, parent Chassis, child LIDAR, origin xyz=0.15 0 0.23 rpy=0 0 0

File: desherborator_description/urdf/desherborator.urdf.xacro (robot description, xacro)
@@ -6,28 +6,4 @@
   <xacro:include filename="$(find desherborator_description)/urdf/desherborator.joint.xacro"/>
   <xacro:include filename="$(find desherborator_description)/urdf/desherborator.sensor.xacro"/>
-  <gazebo>
-    <plugin name="wheels_controller" filename="libgazebo_ros_diff_drive.so">
-      <commandTopic>cmd_vel</commandTopic>
-      <odometryTopic>odom</odometryTopic>
-      <odometryFrame>odom</odometryFrame>
-      <odometrySource>world</odometrySource>
-      <publishOdomTF>true</publishOdomTF>
-      <!-- ENTER BASE LINK NAME -->
-      <robotBaseFrame>base_link</robotBaseFrame>
-      <publishWheelTF>true</publishWheelTF>
-      <publishTf>true</publishTf>
-      <publishWheelJointState>true</publishWheelJointState>
-      <legacyMode>true</legacyMode>
-      <updateRate>30</updateRate>
-      <!-- ENTER LEFT JOINT NAME -->
-      <leftJoint>RoueG</leftJoint>
-      <!-- ENTER RIGHT JOINT NAME -->
-      <rightJoint>RoueD</rightJoint>
-      <wheelSeparation>0.31</wheelSeparation>
-      <wheelDiameter>0.1</wheelDiameter>
-      <wheelAcceleration>0.1</wheelAcceleration>
-      <wheelTorque>10</wheelTorque>
-      <rosDebugLevel>na</rosDebugLevel>
-    </plugin>
-  </gazebo>
+  <xacro:include filename="$(find desherborator_description)/urdf/desherborator.controller.xacro"/>
 </robot>

Commit message: Task 2.11: fix prismatic and revolute joints

File: desherborator_description/urdf/desherborator.joint.xacro (robot description, xacro)
@@ -28,15 +28,17 @@
                 <origin xyz="-0.10 0 0" rpy="0 0 0"/>
         </joint>
-        <joint name="joint_chassis_to_dummy" type="fixed">
+        <joint name="joint_chassis_to_dummy" type="prismatic">
                 <parent link="Chassis"/>
                 <child link="BrasC1dummy"/>
                 <origin xyz="0.19 -0.06 0.2" rpy="0 0 0"/>
                 <axis  xyz="0 0 1"/>
+                <limit upper="1" effort="10" velocity="1" />
         </joint>
-        <joint name="joint_dummy_to_rotating_bras" type="fixed">
+        <joint name="joint_dummy_to_rotating_bras" type="revolute">
                 <parent link="BrasC1dummy"/>
                 <child link="BrasC1"/>
                 <origin xyz="0 0 0" rpy="0 0 0"/>
                 <axis  xyz="0 0 1"/>
+                <limit lower="-3.14" upper="0" effort="10" velocity="1" />
         </joint>
         <joint name="joint_rotating_bras_to_brasS" type="fixed">

File: desherborator_description/urdf/desherborator.link.xacro (robot description, xacro)
@@ -102,5 +102,19 @@
   </link>
   <!-- link Dummy Bras Cylindre 1 -->
-  <link name="BrasC1dummy"/>
+  <link name="BrasC1dummy">
+    <collision>
+      <origin xyz="0 0 0" rpy="0 0 0"/>
+      <geometry>
+        <cylinder radius="0.001" length="0.001"/>
+      </geometry>
+    </collision>
+    <visual>
+      <origin xyz="0 0 0" rpy="0 0 0"/>
+      <geometry>
+        <cylinder radius="0.001" length="0.001"/>
+      </geometry>
+    </visual>
+    <xacro:default_inertial mass="0.001"/>
+  </link>
   <!-- link Bras Cylindre 2 -->
   <link name="BrasC2">

Commit message: Task 4.1 : Bras articulé ( Adding the controller of the arm)

File: desherborator_description/urdf/desherborator.joint.xacro (robot description, xacro)
@@ -31,5 +31,5 @@
                 <parent link="Chassis"/>
                 <child link="BrasC1dummy"/>
-                <origin xyz="0.19 -0.06 0.2" rpy="0 0 0"/>
+                <origin xyz="1 -0.06 0.2" rpy="0 0 0"/>
                 <axis  xyz="0 0 1"/>
                 <limit upper="1" effort="10" velocity="1" />
@@ -62,3 +62,23 @@
                 <origin xyz="0 0 -0.05" rpy="0 0 0"/>
         </joint>
+        <transmission name="trans_sliding_arm">
+                <type>transmission_interface/SimpleTransmission</type>
+                <joint name="joint_chassis_to_dummy">
+                <hardwareInterface>EffortJointInterface</hardwareInterface>
+                </joint>
+                <actuator name="motor_sdiling">
+                <hardwareInterface>EffortJointInterface</hardwareInterface>
+                <mechanicalReduction>1</mechanicalReduction>
+                </actuator>
+        </transmission>
+        <transmission name="trans_rotating_arm">
+                <type>transmission_interface/SimpleTransmission</type>
+                <joint name="joint_dummy_to_rotating_bras">
+                <hardwareInterface>EffortJointInterface</hardwareInterface>
+                </joint>
+                <actuator name="motor_rotating">
+                <hardwareInterface>EffortJointInterface</hardwareInterface>
+                <mechanicalReduction>1</mechanicalReduction>
+                </actuator>
+        </transmission>
 </robot>

File: desherborator_description/urdf/desherborator.urdf.xacro (robot description, xacro)
@@ -6,4 +6,5 @@
   <xacro:include filename="$(find desherborator_description)/urdf/desherborator.joint.xacro"/>
   <xacro:include filename="$(find desherborator_description)/urdf/desherborator.sensor.xacro"/>
-  <xacro:include filename="$(find desherborator_description)/urdf/desherborator.controller.xacro"/>
+  <xacro:include filename="$(find desherborator_description)/urdf/desherborator.wheels_controller.xacro"/>
+  <xacro:include filename="$(find desherborator_description)/urdf/desherborator.arm_controller.xacro"/>
 </robot>

Commit message: Finished Task 4.1 : Bras Articulé

File: desherborator_description/urdf/desherborator.joint.xacro (robot description, xacro)
@@ -31,7 +31,7 @@
                 <parent link="Chassis"/>
                 <child link="BrasC1dummy"/>
-                <origin xyz="1 -0.06 0.2" rpy="0 0 0"/>
+                <origin xyz="0.19 -0.06 0.2" rpy="0 0 0"/>
                 <axis  xyz="0 0 1"/>
-                <limit upper="1" effort="10" velocity="1" />
+                <limit upper="0.1" effort="10" velocity="1" />
         </joint>
         <joint name="joint_dummy_to_rotating_bras" type="revolute">

File: desherborator_description/urdf/desherborator.sensor.xacro (robot description, xacro)
@@ -24,8 +24,8 @@
             <scan>
             <horizontal>
-                <samples>720</samples>
+                <samples>20</samples>
                 <resolution>1</resolution>
-                <min_angle>0.0</min_angle>
-                <max_angle>6.2</max_angle>
+                <min_angle>-3.0</min_angle>
+                <max_angle>3.0</max_angle>
             </horizontal>
             </scan>

Commit message: Task 5.6 Update arm robot size

File: desherborator_description/urdf/desherborator.joint.xacro (robot description, xacro)
@@ -50,10 +50,10 @@
                 <parent link="BrasS1"/>
                 <child link="BrasC2"/>
-                <origin xyz="0 0.15 0" rpy="0  0  0"/>
+                <origin xyz="0 0.2 0" rpy="0  0  0"/>
         </joint>
         <joint name="joint_brasC_to_brasS" type="fixed">
                 <parent link="BrasC2"/>
                 <child link="BrasS2"/>
-                <origin xyz="0 0.15 0" rpy="0 0 0"/>
+                <origin xyz="0 0.2 0" rpy="0 0 0"/>
         </joint>
         <joint name="end_joint" type="fixed">

File: desherborator_description/urdf/desherborator.link.xacro (robot description, xacro)
@@ -128,5 +128,5 @@
       <origin xyz="0 0 0" rpy="0 ${PI/2} ${PI/2}"/>
       <geometry>
-        <cylinder radius="0.01" length="0.3"/>
+        <cylinder radius="0.01" length="0.4"/>
       </geometry>
     </visual>
